File: pcb/vanillaice40/vanillaice40.kicad_pcb (KiCad board)
At the start: 4 copper layers, 100 x 62 mm, 109 parts, among them J1 FX18-120S-0.8SV20, J2 SM04B-SRSS-TBLFSN, J3 Conn_01x02_Pin, SW1 USR1, SW2 USR1, SW3 RESET, U1 TPS563252DRLR, U2 ICE40HX4K-TQ144, U3 W25X40CLSN, U4 TPS563252DRLR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

Commit message: undo ice40 routing
Parts:
- moved R32 4.89 mm to (88.4, 64.1)
- moved R33 4.07 mm to (89.2, 62.6)
- moved C10 2.67 mm to (103.4, 49.0)
- moved R4 2.34 mm to (106.7, 44.7)
- moved C8 1.40 mm to (102.9, 74.0)
- moved C28 1.40 mm to (105.1, 74.0)
- moved C29 0.76 mm to (99.2, 74.5)
- moved C12 0.61 mm to (112.6, 74.0), turned to 0 degrees
Routing:
- net /IOL_3B: track 66.0 -> 0.00 mm
- net /IOL_3A: track 65.5 -> 0.00 mm
- net /IOL_2B: track 64.9 -> 0.00 mm
- net /IOL_2A: track 64.0 -> 0.00 mm
- net /IOT_214: track 63.3 -> 0.00 mm
- net /IOT_213: track 63.2 -> 0.00 mm
- net /IOT_212: track 63.2 -> 0.00 mm
- net /IOT_219: track 63.1 -> 0.00 mm
- net /IOT_215: track 63.1 -> 0.00 mm
- net /IOT_217: track 63.1 -> 0.00 mm
- net /IOT_216: track 63.1 -> 0.00 mm
- net /IOT_198: track 62.7 -> 0.00 mm, vias 2 -> 0
- net /IOT_197: track 61.9 -> 0.00 mm, vias 2 -> 0
- net /IOT_191: track 60.9 -> 0.00 mm
- net /IOT_222: track 60.7 -> 0.00 mm
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
Commit message: io moved to lower diff
Connections:
- J1 pad 10: /IOR_148 -> unconnected-(J1-Pad10)
- J1 pad 100: /IOT_206 -> unconnected-(J1-Pad100)
- J1 pad 101: +3V3 -> unconnected-(J1-Pad101)
- J1 pad 102: GND -> unconnected-(J1-Pad102)
- J1 pad 103: /IOT_198 -> unconnected-(J1-Pad103)
- J1 pad 104: /IOT_197 -> unconnected-(J1-Pad104)
- J1 pad 105: /IOT_192 -> unconnected-(J1-Pad105)
- J1 pad 106: /IOT_191 -> unconnected-(J1-Pad106)
- J1 pad 107: /IOT_190 -> unconnected-(J1-Pad107)
- J1 pad 108: /IOT_181 -> unconnected-(J1-Pad108)
- J1 pad 109: /IOT_179 -> unconnected-(J1-Pad109)
- J1 pad 11: +3V3 -> unconnected-(J1-Pad11)
- J1 pad 110: GND -> unconnected-(J1-Pad110)
- J1 pad 111: /IOT_178 -> unconnected-(J1-Pad111)
- J1 pad 112: /IOT_177 -> unconnected-(J1-Pad112)
- J1 pad 113: /IOT_174 -> unconnected-(J1-Pad113)
- J1 pad 114: /IOT_173 -> unconnected-(J1-Pad114)
- J1 pad 115: /IOT_172 -> unconnected-(J1-Pad115)
- J1 pad 116: /IOT_171 -> unconnected-(J1-Pad116)
- J1 pad 117: /IOT_170 -> unconnected-(J1-Pad117)
- J1 pad 118: /IOT_169 -> unconnected-(J1-Pad118)
- J1 pad 119: /IOT_168 -> unconnected-(J1-Pad119)
- J1 pad 12: GND -> unconnected-(J1-Pad12)
- J1 pad 120: GND -> unconnected-(J1-Pad120)
- J1 pad 13: /IOR_147 -> unconnected-(J1-Pad13)
- J1 pad 14: /IOR_146 -> unconnected-(J1-Pad14)
- J1 pad 15: /IOR_144 -> unconnected-(J1-Pad15)
- J1 pad 16: /IOR_141 -> unconnected-(J1-Pad16)
- J1 pad 17: /IOR_140 -> unconnected-(J1-Pad17)
- J1 pad 18: /IOR_139 -> unconnected-(J1-Pad18)
- J1 pad 19: /IOR_138 -> unconnected-(J1-Pad19)
- J1 pad 20: GND -> unconnected-(J1-Pad20)
- J1 pad 21: +3V3 -> unconnected-(J1-Pad21)
- J1 pad 22: GND -> unconnected-(J1-Pad22)
- J1 pad 23: /IOR_137 -> unconnected-(J1-Pad23)
- J1 pad 24: /IOR_136 -> unconnected-(J1-Pad24)
- J1 pad 25: /IOR_128 -> unconnected-(J1-Pad25)
- J1 pad 26: /IOR_120 -> unconnected-(J1-Pad26)
- J1 pad 27: /IOR_119 -> unconnected-(J1-Pad27)
- J1 pad 28: /IOR_118 -> unconnected-(J1-Pad28)
- J1 pad 29: /IOR_117 -> unconnected-(J1-Pad29)
- J1 pad 3: /IOR_167 -> unconnected-(J1-Pad3)
- J1 pad 30: GND -> unconnected-(J1-Pad30)
- J1 pad 31: +3V3 -> unconnected-(J1-Pad31)
- J1 pad 32: GND -> unconnected-(J1-Pad32)
- J1 pad 33: /IOR_116 -> unconnected-(J1-Pad33)
- J1 pad 34: /IOR_115 -> unconnected-(J1-Pad34)
- J1 pad 35: /IOR_114 -> unconnected-(J1-Pad35)
- J1 pad 36: /IOR_112 -> unconnected-(J1-Pad36)
- J1 pad 37: /IOR_111 -> unconnected-(J1-Pad37)
- J1 pad 38: /IOR_110 -> unconnected-(J1-Pad38)
- J1 pad 39: /IOR_109 -> unconnected-(J1-Pad39)
- J1 pad 4: /IOR_166 -> unconnected-(J1-Pad4)
- J1 pad 40: /IOB_102 -> unconnected-(J1-Pad40)
- J1 pad 41: +3V3 -> unconnected-(J1-Pad41)
- J1 pad 42: GND -> unconnected-(J1-Pad42)
- J1 pad 43: /IOB_96 -> unconnected-(J1-Pad43)
- J1 pad 44: /IOB_95 -> unconnected-(J1-Pad44)
- J1 pad 45: /IOB_94 -> unconnected-(J1-Pad45)
- J1 pad 46: /IOB_91 -> unconnected-(J1-Pad46)
- J1 pad 47: /IOB_82 -> unconnected-(J1-Pad47)
- J1 pad 48: /IOB_81 -> unconnected-(J1-Pad48)
- J1 pad 49: /IOB_80 -> unconnected-(J1-Pad49)
- J1 pad 5: /IOR_165 -> unconnected-(J1-Pad5)
- J1 pad 50: GND -> unconnected-(J1-Pad50)
- J1 pad 51: /IOB_79 -> unconnected-(J1-Pad51)
- J1 pad 52: /IOB_73 -> unconnected-(J1-Pad52)
- J1 pad 53: /IOB_72 -> unconnected-(J1-Pad53)
- J1 pad 54: /IOB_71 -> unconnected-(J1-Pad54)
- J1 pad 55: /IOB_64 -> unconnected-(J1-Pad55)
- J1 pad 56: /IOB_63 -> unconnected-(J1-Pad56)
- J1 pad 57: /IOB_61 -> unconnected-(J1-Pad57)
- J1 pad 58: /IOB_57 -> unconnected-(J1-Pad58)
- J1 pad 59: /IOB_56 -> unconnected-(J1-Pad59)
- J1 pad 6: /IOR_164 -> unconnected-(J1-Pad6)
- J1 pad 60: GND -> unconnected-(J1-Pad60)
- J1 pad 63: /IOL_17B -> unconnected-(J1-Pad63)
- J1 pad 64: /IOL_17A -> unconnected-(J1-Pad64)
- J1 pad 65: /IOL_14B -> unconnected-(J1-Pad65)
- J1 pad 66: /IOL_13B -> unconnected-(J1-Pad66)
- J1 pad 67: /IOL_13A -> unconnected-(J1-Pad67)
- J1 pad 68: /IOL_12B -> unconnected-(J1-Pad68)
- J1 pad 69: /IOL_12A -> unconnected-(J1-Pad69)
- J1 pad 7: /IOR_161 -> unconnected-(J1-Pad7)
- J1 pad 70: /IOL_10B -> unconnected-(J1-Pad70)
- J1 pad 71: +3V3 -> unconnected-(J1-Pad71)
- J1 pad 72: GND -> unconnected-(J1-Pad72)
- J1 pad 73: /IOL_10A -> unconnected-(J1-Pad73)
- J1 pad 74: /IOL_8B -> unconnected-(J1-Pad74)
- J1 pad 75: /IOL_8A -> unconnected-(J1-Pad75)
- J1 pad 76: /IOL_5B -> unconnected-(J1-Pad76)
- J1 pad 77: /IOL_5A -> unconnected-(J1-Pad77)
- J1 pad 78: /IOL_4B -> unconnected-(J1-Pad78)
- J1 pad 79: /IOL_4A -> unconnected-(J1-Pad79)
- J1 pad 8: /IOR_160 -> unconnected-(J1-Pad8)
- J1 pad 80: GND -> unconnected-(J1-Pad80)
- J1 pad 81: +3V3 -> unconnected-(J1-Pad81)
- J1 pad 82: GND -> unconnected-(J1-Pad82)
- J1 pad 83: /IOL_3B -> unconnected-(J1-Pad83)
- J1 pad 84: /IOL_3A -> unconnected-(J1-Pad84)
- J1 pad 85: /IOL_2B -> unconnected-(J1-Pad85)
- J1 pad 86: /IOL_2A -> unconnected-(J1-Pad86)
- J1 pad 87: /IOT_222 -> unconnected-(J1-Pad87)
- J1 pad 88: /IOT_221 -> unconnected-(J1-Pad88)
- J1 pad 89: /IOT_220 -> unconnected-(J1-Pad89)
- J1 pad 9: /IOR_152 -> unconnected-(J1-Pad9)
- J1 pad 90: GND -> unconnected-(J1-Pad90)
- J1 pad 91: +3V3 -> unconnected-(J1-Pad91)
- J1 pad 92: GND -> unconnected-(J1-Pad92)
- J1 pad 93: /IOT_219 -> unconnected-(J1-Pad93)
- J1 pad 94: /IOT_217 -> unconnected-(J1-Pad94)
- J1 pad 95: /IOT_216 -> unconnected-(J1-Pad95)
- J1 pad 96: /IOT_215 -> unconnected-(J1-Pad96)
- J1 pad 97: /IOT_214 -> unconnected-(J1-Pad97)
- J1 pad 98: /IOT_213 -> unconnected-(J1-Pad98)
- J1 pad 99: /IOT_212 -> unconnected-(J1-Pad99)
- J2 pad 1: /IOL_23A -> /IOL_5A
- J2 pad 2: /IOL_23B -> /IOL_5B
- R1 pad 1: /IOL_24A -> /IOL_2A
- R2 pad 1: /IOL_24B -> /IOL_2B
- R32 pad 2: /IOL_25A -> /IOL_4A
- R33 pad 2: /IOL_25B -> /IOL_4B
- R7 pad 2: /IOL_18A -> /IOL_3A
- R8 pad 2: /IOL_18B -> /IOL_3B
- SW1 pad 2: /IOL_18A -> /IOL_3A
- SW2 pad 2: /IOL_18B -> /IOL_3B

Commit message: fx18 power redo
Connections:
- J1 pad 100: unconnected-(J1-Pad100) -> GND
- J1 pad 109: unconnected-(J1-Pad109) -> +3V3
- J1 pad 11: unconnected-(J1-Pad11) -> +3V3
- J1 pad 110: unconnected-(J1-Pad110) -> GND
- J1 pad 119: unconnected-(J1-Pad119) -> +3V3
- J1 pad 12: unconnected-(J1-Pad12) -> GND
- J1 pad 120: unconnected-(J1-Pad120) -> GND
- J1 pad 21: unconnected-(J1-Pad21) -> +3V3
- J1 pad 22: unconnected-(J1-Pad22) -> GND
- J1 pad 39: unconnected-(J1-Pad39) -> +3V3
- J1 pad 40: unconnected-(J1-Pad40) -> GND
- J1 pad 49: unconnected-(J1-Pad49) -> +3V3
- J1 pad 50: unconnected-(J1-Pad50) -> GND
- J1 pad 59: unconnected-(J1-Pad59) -> +3V3
- J1 pad 60: unconnected-(J1-Pad60) -> GND
- J1 pad 70: unconnected-(J1-Pad70) -> +3V3
- J1 pad 71: unconnected-(J1-Pad71) -> GND
- J1 pad 80: unconnected-(J1-Pad80) -> +3V3
- J1 pad 81: unconnected-(J1-Pad81) -> GND
- J1 pad 99: unconnected-(J1-Pad99) -> +3V3

Commit message: start of 3rd reroute
Parts:
- removed R7, R8: 10k, Resistor_SMD:R_0603_1608Metric
- removed SW1, SW2: USR1, Button_Switch_SMD:SW_SPST_PTS810
Connections:
- J1 pad 10: unconnected-(J1-Pad10) -> /IOT_179
- J1 pad 101: unconnected-(J1-Pad101) -> /IOB_96
- J1 pad 102: unconnected-(J1-Pad102) -> /IOB_95
- J1 pad 103: unconnected-(J1-Pad103) -> /IOB_94
- J1 pad 104: unconnected-(J1-Pad104) -> /IOB_91
- J1 pad 105: unconnected-(J1-Pad105) -> /IOB_82
- J1 pad 106: unconnected-(J1-Pad106) -> /IOB_81
- J1 pad 107: unconnected-(J1-Pad107) -> /IOB_80
- J1 pad 108: unconnected-(J1-Pad108) -> /IOB_79
- J1 pad 111: unconnected-(J1-Pad111) -> /IOB_73
- J1 pad 112: unconnected-(J1-Pad112) -> /IOB_72
- J1 pad 113: unconnected-(J1-Pad113) -> /IOB_71
- J1 pad 114: unconnected-(J1-Pad114) -> /IOB_64
- J1 pad 115: unconnected-(J1-Pad115) -> /IOB_63
- J1 pad 116: unconnected-(J1-Pad116) -> /IOB_61
- J1 pad 117: unconnected-(J1-Pad117) -> /IOB_57
- J1 pad 118: unconnected-(J1-Pad118) -> /IOB_56
- J1 pad 13: unconnected-(J1-Pad13) -> /IOT_181
- J1 pad 14: unconnected-(J1-Pad14) -> /IOT_190
- J1 pad 15: unconnected-(J1-Pad15) -> /IOT_191
- J1 pad 16: unconnected-(J1-Pad16) -> /IOT_192
- J1 pad 17: unconnected-(J1-Pad17) -> /IOT_197
- J1 pad 18: unconnected-(J1-Pad18) -> /IOT_198
- J1 pad 19: unconnected-(J1-Pad19) -> /IOT_206
- J1 pad 20: unconnected-(J1-Pad20) -> /IOT_212
- J1 pad 23: unconnected-(J1-Pad23) -> /IOT_213
- J1 pad 24: unconnected-(J1-Pad24) -> /IOT_214
- J1 pad 25: unconnected-(J1-Pad25) -> /IOT_215
- J1 pad 26: unconnected-(J1-Pad26) -> /IOT_216
- J1 pad 27: unconnected-(J1-Pad27) -> /IOT_217
- J1 pad 28: unconnected-(J1-Pad28) -> /IOT_219
- J1 pad 29: unconnected-(J1-Pad29) -> /IOT_220
- J1 pad 3: unconnected-(J1-Pad3) -> /IOT_170
- J1 pad 30: unconnected-(J1-Pad30) -> /IOT_221
- J1 pad 31: unconnected-(J1-Pad31) -> /IOT_222
- J1 pad 32: unconnected-(J1-Pad32) -> /IOL_4A
- J1 pad 33: unconnected-(J1-Pad33) -> /IOL_4B
- J1 pad 34: unconnected-(J1-Pad34) -> /IOL_5A
- J1 pad 35: unconnected-(J1-Pad35) -> /IOL_5B
- J1 pad 36: unconnected-(J1-Pad36) -> /IOL_8A
- J1 pad 37: unconnected-(J1-Pad37) -> /IOL_8B
- J1 pad 38: unconnected-(J1-Pad38) -> /IOL_10A
- J1 pad 4: unconnected-(J1-Pad4) -> /IOT_171
- J1 pad 41: unconnected-(J1-Pad41) -> /IOL_10B
- J1 pad 42: unconnected-(J1-Pad42) -> /IOL_12A
- J1 pad 43: unconnected-(J1-Pad43) -> /IOL_12B
- J1 pad 44: unconnected-(J1-Pad44) -> /IOL_13A
- J1 pad 45: unconnected-(J1-Pad45) -> /IOL_13B
- J1 pad 46: unconnected-(J1-Pad46) -> /IOL_14B
- J1 pad 47: unconnected-(J1-Pad47) -> /IOL_17A
- J1 pad 48: unconnected-(J1-Pad48) -> /IOL_17B
- J1 pad 5: unconnected-(J1-Pad5) -> /IOT_172
- J1 pad 51: unconnected-(J1-Pad51) -> /IOL_18A
- J1 pad 52: unconnected-(J1-Pad52) -> /IOL_18B
- J1 pad 53: unconnected-(J1-Pad53) -> /IOL_23A
- J1 pad 54: unconnected-(J1-Pad54) -> /IOL_23B
- J1 pad 55: unconnected-(J1-Pad55) -> /IOL_24A
- J1 pad 56: unconnected-(J1-Pad56) -> /IOL_24B
- J1 pad 57: unconnected-(J1-Pad57) -> /IOL_25A
- J1 pad 58: unconnected-(J1-Pad58) -> /IOL_25B
- J1 pad 6: unconnected-(J1-Pad6) -> /IOT_173
- J1 pad 63: unconnected-(J1-Pad63) -> /IOT_169
- J1 pad 64: unconnected-(J1-Pad64) -> /IOT_168
- J1 pad 65: unconnected-(J1-Pad65) -> /IOR_167
- J1 pad 66: unconnected-(J1-Pad66) -> /IOR_166
- J1 pad 67: unconnected-(J1-Pad67) -> /IOR_165
- J1 pad 68: unconnected-(J1-Pad68) -> /IOR_164
- J1 pad 69: unconnected-(J1-Pad69) -> /IOR_161
- J1 pad 7: unconnected-(J1-Pad7) -> /IOT_174
- J1 pad 72: unconnected-(J1-Pad72) -> /IOR_160
- J1 pad 73: unconnected-(J1-Pad73) -> /IOR_152
- J1 pad 74: unconnected-(J1-Pad74) -> /IOR_148
- J1 pad 75: unconnected-(J1-Pad75) -> /IOR_147
- J1 pad 76: unconnected-(J1-Pad76) -> /IOR_146
- J1 pad 77: unconnected-(J1-Pad77) -> /IOR_144
- J1 pad 78: unconnected-(J1-Pad78) -> /IOR_141
- J1 pad 79: unconnected-(J1-Pad79) -> /IOR_140
- J1 pad 8: unconnected-(J1-Pad8) -> /IOT_177
- J1 pad 82: unconnected-(J1-Pad82) -> /IOR_139
- J1 pad 83: unconnected-(J1-Pad83) -> /IOR_138
- J1 pad 84: unconnected-(J1-Pad84) -> /IOR_137
- J1 pad 85: unconnected-(J1-Pad85) -> /IOR_136
- J1 pad 86: unconnected-(J1-Pad86) -> /IOR_128
- J1 pad 87: unconnected-(J1-Pad87) -> /IOR_120
- J1 pad 88: unconnected-(J1-Pad88) -> /IOR_119
- J1 pad 89: unconnected-(J1-Pad89) -> /IOR_118
- J1 pad 9: unconnected-(J1-Pad9) -> /IOT_178
- J1 pad 90: unconnected-(J1-Pad90) -> /IOR_117
- J1 pad 91: unconnected-(J1-Pad91) -> /IOR_116
- J1 pad 92: unconnected-(J1-Pad92) -> /IOR_115
- J1 pad 93: unconnected-(J1-Pad93) -> /IOR_114
- J1 pad 94: unconnected-(J1-Pad94) -> /IOR_112
- J1 pad 95: unconnected-(J1-Pad95) -> /IOR_111
- J1 pad 96: unconnected-(J1-Pad96) -> /IOR_110
- J1 pad 97: unconnected-(J1-Pad97) -> /IOR_109
- J1 pad 98: unconnected-(J1-Pad98) -> /IOB_102
- J2 pad 1: /IOL_5A -> /IOL_4A
- J2 pad 2: /IOL_5B -> /IOL_4B
- R32 pad 2: /IOL_4A -> /IOL_3A
- R33 pad 2: /IOL_4B -> /IOL_3B

Commit message: connector vias
Routing:
- net +3V3: track 75.2 -> 96.1 mm, vias 20 -> 32
- net GND: track 79.6 -> 100.5 mm, vias 57 -> 85
- net /IOL_25B: track 0.00 -> 2.94 mm, vias 0 -> 2
- net /IOL_8A: track 0.05 -> 1.79 mm, vias 0 -> 1
- net /IOL_24A: track 0.00 -> 1.74 mm, vias 0 -> 1
- net /IOL_23B: track 0.00 -> 1.74 mm, vias 0 -> 1
- net /IOL_23A: track 0.00 -> 1.74 mm, vias 0 -> 1
- net /IOL_13B: track 0.00 -> 1.74 mm, vias 0 -> 1
- net /IOL_13A: track 0.00 -> 1.74 mm, vias 0 -> 1
- net /IOL_12A: track 0.00 -> 1.74 mm, vias 0 -> 1
- net /IOL_10B: track 0.00 -> 1.74 mm, vias 0 -> 1
- net /IOT_222: track 0.00 -> 1.74 mm, vias 0 -> 1
- net /IOT_221: track 0.00 -> 1.74 mm, vias 0 -> 1
- net /IOT_220: track 0.00 -> 1.74 mm, vias 0 -> 1
- net /IOT_219: track 0.00 -> 1.74 mm, vias 0 -> 1
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
Commit message: iol redone
Parts:
- moved C3 27.3 mm to (90.0, 53.7), turned to 180 degrees
Routing:
- net /IOL_24B: track 1.74 -> 56.4 mm, vias 1 -> 2
- net /IOL_23B: track 1.74 -> 56.3 mm, vias 1 -> 2
- net /IOL_18B: track 1.74 -> 56.3 mm, vias 1 -> 2
- net /IOL_4A: track 1.74 -> 55.9 mm, vias 1 -> 2
- net /IOL_17B: track 1.74 -> 55.5 mm, vias 1 -> 2
- net /IOL_14B: track 1.74 -> 55.3 mm, vias 1 -> 2
- net /IOL_5A: track 1.74 -> 55.3 mm, vias 1 -> 2
- net /IOL_13A: track 1.74 -> 55.2 mm, vias 1 -> 2
- net /IOL_12A: track 1.74 -> 55.0 mm, vias 1 -> 2
- net /IOL_8A: track 1.79 -> 54.7 mm, vias 1 -> 2
- net /IOL_10A: track 1.74 -> 54.1 mm, vias 1 -> 2
- net /IOL_25A: track 1.74 -> 53.8 mm, vias 1 -> 2
- net /IOL_24A: track 1.74 -> 53.5 mm, vias 1 -> 2
- net /IOL_18A: track 1.74 -> 53.4 mm, vias 1 -> 3
- net /IOL_23A: track 1.74 -> 53.4 mm, vias 1 -> 2
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- added copper zone on B.Cu, net GND
- added copper zone on F.Cu, net GND

Commit message: iob redone
Routing:
- net /IOB_61: track 0.00 -> 48.0 mm, vias 0 -> 2
- net /IOB_56: track 0.00 -> 47.3 mm
- net /IOB_57: track 0.00 -> 46.6 mm
- net /IOB_72: track 0.00 -> 45.6 mm, vias 0 -> 2
- net /IOB_63: track 0.00 -> 44.3 mm
- net /IOB_73: track 0.00 -> 44.2 mm, vias 0 -> 2
- net /IOB_64: track 0.00 -> 43.5 mm
- net /IOB_71: track 0.00 -> 43.0 mm
- net /IOB_79: track 0.00 -> 39.0 mm, vias 0 -> 2
- net /IOB_80: track 0.00 -> 38.8 mm, vias 0 -> 2
- net /IOB_81: track 0.00 -> 37.4 mm, vias 0 -> 2
- net /IOB_82: track 0.00 -> 35.0 mm, vias 0 -> 2
- net /IOB_91: track 0.00 -> 33.6 mm, vias 0 -> 2
- net GND: track 120.8 -> 112.1 mm, vias 94 -> 89
- net +3V3: track 96.1 -> 87.4 mm, vias 32 -> 27
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
Commit message: final rough draft
Parts:
- added C44: 0.1uf, Capacitor_SMD:C_0402_1005Metric, F.Cu at (116.5, 60.8)
Connections:
- J1 pad 10: /IOT_179 -> /IOT_181
- J1 pad 13: /IOT_181 -> /IOT_179
- J1 pad 14: /IOT_190 -> /IOT_178
- J1 pad 15: /IOT_191 -> /IOT_177
- J1 pad 16: /IOT_192 -> /IOT_174
- J1 pad 17: /IOT_197 -> /IOT_173
- J1 pad 18: /IOT_198 -> /IOT_172
- J1 pad 19: /IOT_206 -> /IOT_171
- J1 pad 20: /IOT_212 -> /IOT_170
- J1 pad 3: /IOT_170 -> /IOT_212
- J1 pad 4: /IOT_171 -> /IOT_206
- J1 pad 5: /IOT_172 -> /IOT_198
- J1 pad 6: /IOT_173 -> /IOT_197
- J1 pad 7: /IOT_174 -> /IOT_192
- J1 pad 8: /IOT_177 -> /IOT_191
- J1 pad 9: /IOT_178 -> /IOT_190
Routing:
- net /IOT_221: track 0.00 -> 53.9 mm, vias 0 -> 2
- net /IOT_219: track 0.00 -> 52.5 mm, vias 0 -> 2
- net /IOT_222: track 0.00 -> 52.2 mm, vias 0 -> 2
- net /IOT_216: track 0.00 -> 50.5 mm, vias 0 -> 2
- net /IOT_220: track 0.00 -> 50.5 mm, vias 0 -> 2
- net /IOT_217: track 0.00 -> 48.9 mm, vias 0 -> 2
- net /IOT_214: track 0.00 -> 48.4 mm, vias 0 -> 2
- net /IOT_206: track 0.00 -> 48.4 mm, vias 0 -> 2
- net /IOT_215: track 0.00 -> 47.0 mm, vias 0 -> 2
- net /IOT_212: track 0.00 -> 46.5 mm, vias 0 -> 2
- net /IOT_197: track 0.00 -> 46.3 mm, vias 0 -> 2
- net /IOT_213: track 0.00 -> 44.9 mm, vias 0 -> 2
- net /IOT_191: track 0.00 -> 44.3 mm, vias 0 -> 2
- net /IOT_198: track 0.00 -> 44.1 mm, vias 0 -> 2
- net /IOT_181: track 0.00 -> 43.8 mm, vias 0 -> 2
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