File: pcb/vanillaice40/vanillaice40.kicad_sch (KiCad schematic)
At the start: 105 parts, among them J1 FX18-120S-0.8SV20, J2 SM04B-SRSS-TBLFSN, J3 Conn_01x02_Pin, SW3 RESET, U1 TPS563252DRLR, U2 ICE40HX4K-TQ144, U3 W25X40CLSN, U4 TPS563252DRLR, U5 FT2232HL, U6 93LCxxBxxOT, X1 SG-8101CE 100Mhz, Y1 12Mhz/18pf

Commit message: final rough draft
Parts:
- added C44: 0.1uf, Capacitor_SMD:C_0402_1005Metric, symbol Device:C_Small
Connections:
- net +1V2: now also C44.1
- net GND: now also C44.2
- net IOT_170: now also J1.20; no longer J1.3
- net IOT_171: now also J1.19; no longer J1.4
- net IOT_172: now also J1.18; no longer J1.5
- net IOT_173: now also J1.17; no longer J1.6
- net IOT_174: now also J1.16; no longer J1.7
- net IOT_177: now also J1.15; no longer J1.8
- net IOT_178: now also J1.14; no longer J1.9
- net IOT_179: now also J1.13; no longer J1.10
- net IOT_181: now also J1.10; no longer J1.13
- net IOT_190: now also J1.9; no longer J1.14
- net IOT_191: now also J1.8; no longer J1.15
- net IOT_192: now also J1.7; no longer J1.16
- net IOT_197: now also J1.6; no longer J1.17
- net IOT_198: now also J1.5; no longer J1.18
- net IOT_206: now also J1.4; no longer J1.19
- net IOT_212: now also J1.3; no longer J1.20
Other:
- moved on the sheet: C2
Changed lines of the file:
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@@
 	)
 	(junction
+		(at 288.29 38.1)
+		(diameter 0)
+		(color 0 0 0 0)
+	)
+	(junction
 		(at 342.9 137.16)
 		(diameter 0)
@@
 	)
 	(junction
+		(at 288.29 27.94)
+		(diameter 0)
+		(color 0 0 0 0)
+	)
+	(junction
 		(at 375.92 49.53)
 		(diameter 0)
@@
 	(wire
 		(pts
-			(xy 288.29 30.48) (xy 288.29 27.94)
+			(xy 278.13 30.48) (xy 278.13 27.94)
 		)
 		(stroke
@@
 	(wire
 		(pts
-			(xy 288.29 38.1) (xy 298.45 38.1)
+			(xy 278.13 38.1) (xy 288.29 38.1)
 		)
 		(stroke
@@
 	(wire
 		(pts
+			(xy 288.29 35.56) (xy 288.29 38.1)
+		)
+		(stroke
+			(width 0)
+			(type default)
+		)
+	)
+	(wire
+		(pts
 			(xy 53.34 58.42) (xy 50.8 58.42)
 		)
@@
 	(wire
 		(pts
+			(xy 288.29 38.1) (xy 298.45 38.1)
+		)
+		(stroke
+			(width 0)
+			(type default)
+		)
+	)
+	(wire
+		(pts
 			(xy 227.33 226.06) (xy 237.49 226.06)
 		)
@@
 	(wire
 		(pts
+			(xy 288.29 27.94) (xy 288.29 30.48)
+		)
+		(stroke
+			(width 0)
+			(type default)
+		)
+	)
+	(wire
+		(pts
 			(xy 67.31 45.72) (xy 67.31 58.42)
 		)
@@
 	(wire
 		(pts
-			(xy 288.29 35.56) (xy 288.29 38.1)
+			(xy 278.13 35.56) (xy 278.13 38.1)
 		)
 		(stroke
@@
 	(wire
 		(pts
-			(xy 288.29 27.94) (xy 298.45 27.94)
+			(xy 278.13 27.94) (xy 288.29 27.94)
 		)
 		(stroke
@@
 	(wire
 		(pts
+			(xy 288.29 27.94) (xy 298.45 27.94)
+		)
+		(stroke
+			(width 0)
+			(type default)
+		)
+	)
+	(wire
+		(pts
 			(xy 81.28 177.8) (xy 81.28 185.42)
 		)
@@
 	)
 	(label "IOT_179"
-		(at 201.93 170.18 0)
+		(at 201.93 177.8 0)
 		(fields_autoplaced yes)
 		(effects
@@
 	)
 	(label "IOT_170"
-		(at 201.93 152.4 0)
+		(at 201.93 195.58 0)
 		(fields_autoplaced yes)
 		(effects
@@
 	)
 	(label "IOT_171"
-		(at 201.93 154.94 0)
+		(at 201.93 193.04 0)
 		(fields_autoplaced yes)
 		(effects
@@
 	)
 	(label "IOT_191"
-		(at 201.93 182.88 0)
+		(at 201.93 165.1 0)
 		(fields_autoplaced yes)
 		(effects
@@
 	)
 	(label "IOT_174"
-		(at 201.93 162.56 0)
+		(at 201.93 185.42 0)
 		(fields_autoplaced yes)
 		(effects
@@
 	)
 	(label "IOT_177"
-		(at 201.93 165.1 0)
+		(at 201.93 182.88 0)
 		(fields_autoplaced yes)
 		(effects
@@
 	)
 	(label "IOT_190"
-		(at 201.93 180.34 0)
+		(at 201.93 167.64 0)
 		(fields_autoplaced yes)
 		(effects
@@
 	)
 	(label "IOT_173"
-		(at 201.93 160.02 0)
+		(at 201.93 187.96 0)
 		(fields_autoplaced yes)
 		(effects
@@
 	)
 	(label "IOT_212"
-		(at 201.93 195.58 0)
+		(at 201.93 152.4 0)
 		(fields_autoplaced yes)
 		(effects
@@
 	)
 	(label "IOT_206"
-		(at 201.93 193.04 0)
+		(at 201.93 154.94 0)
 		(fields_autoplaced yes)
 		(effects
@@
 	)
 	(label "IOT_172"
-		(at 201.93 157.48 0)
+		(at 201.93 190.5 0)
 		(fields_autoplaced yes)
 		(effects
@@
 	)
 	(label "IOT_178"
-		(at 201.93 167.64 0)
+		(at 201.93 180.34 0)
 		(fields_autoplaced yes)
 		(effects
@@
 	)
 	(label "IOT_198"
-		(at 201.93 190.5 0)
+		(at 201.93 157.48 0)
 		(fields_autoplaced yes)
 		(effects
@@
 	)
 	(label "IOT_181"
-		(at 201.93 177.8 0)
+		(at 201.93 170.18 0)
 		(fields_autoplaced yes)
 		(effects
@@
 	)
 	(label "IOT_197"
-		(at 201.93 187.96 0)
+		(at 201.93 160.02 0)
 		(fields_autoplaced yes)
 		(effects
@@
 	)
 	(label "IOT_192"
-		(at 201.93 185.42 0)
+		(at 201.93 162.56 0)
 		(fields_autoplaced yes)
 		(effects
@@
 	)
 	(symbol
+		(lib_id "Device:C_Small")
+		(at 288.29 33.02 0)
+		(unit 1)
+		(exclude_from_sim no)
+		(in_bom yes)
+		(on_board yes)
+		(dnp no)
+		(fields_autoplaced yes)
+		(property "Reference" "C44"
+			(at 290.83 31.7562 0)
+			(effects
+				(font
+					(size 1.27 1.27)
+				)
+				(justify left)
+			)
+		)
+		(property "Value" "0.1uf"
+			(at 290.83 34.2962 0)
+			(effects
+				(font
+					(size 1.27 1.27)
+				)
+				(justify left)
+			)
+		)
+		(property "Footprint" "Capacitor_SMD:C_0402_1005Metric"
+			(at 288.29 33.02 0)
+			(effects
+				(font
+					(size 1.27 1.27)
+				)
+				(hide yes)
+			)
+		)
+		(property "Datasheet" "~"
+			(at 288.29 33.02 0)
+			(effects
+				(font
+					(size 1.27 1.27)
+				)
+				(hide yes)
+			)
+		)
+		(property "Description" "Unpolarized capacitor, small symbol"
+			(at 288.29 33.02 0)
+			(effects
+				(font
+					(size 1.27 1.27)
+				)
+				(hide yes)
+			)
+		)
+		(property "MFG_Part" ""
+			(at 288.29 33.02 0)
+			(effects
+				(font
+					(size 1.27 1.27)
+				)
+				(hide yes)
+			)
+		)
+		(pin "2"
+		)
+		(pin "1"
+		)
+		(instances
+			(project "vanillaice40"
+				(path "/a9f93d6d-ad6a-4eb5-8259-93de27758801"
+					(reference "C44")
+					(unit 1)
+				)
+			)
+		)
+	)
+	(symbol
 		(lib_id "Device:R_Small")
 		(at 254 120.65 180)
@@
 	(symbol
 		(lib_id "Device:C_Small")
-		(at 288.29 33.02 0)
+		(at 278.13 33.02 0)
 		(unit 1)
 		(exclude_from_sim no)
@@
 		(fields_autoplaced yes)
 		(property "Reference" "C2"
-			(at 290.83 31.7562 0)
+			(at 280.67 31.7562 0)
 			(effects
 				(font
@@
 		)
 		(property "Value" "22uf"
-			(at 290.83 34.2962 0)
+			(at 280.67 34.2962 0)
 			(effects
 				(font
@@
 		)
 		(property "Footprint" "Capacitor_SMD:C_0603_1608Metric"
-			(at 288.29 33.02 0)
+			(at 278.13 33.02 0)
 			(effects
 				(font
@@
 		)
 		(property "Datasheet" "~"
-			(at 288.29 33.02 0)
+			(at 278.13 33.02 0)
 			(effects
 				(font
@@
 		)
 		(property "Description" "Unpolarized capacitor, small symbol"
-			(at 288.29 33.02 0)
+			(at 278.13 33.02 0)
 			(effects
 				(font
@@
 		)
 		(property "MFG_Part" ""
-			(at 288.29 33.02 0)
+			(at 278.13 33.02 0)
 			(effects
 				(font
