File: pcb/vanillaice40/vanillaice40.kicad_sch (KiCad schematic)
At the start: 109 parts, among them J1 Conn_01x02_Pin, J2 SM04B-SRSS-TBLFSN, J3 FX18-120S-0.8SV20, J4 Conn_01x06_Pin, J5 Conn_01x02_Pin, J6 Conn_01x02_Pin, J7 Conn_01x02_Pin, U1 TPS563252DRLR, U2 ICE40HX4K-TQ144, U3 W25X40CLSN, U4 TPS563252DRLR, U5 FT2232HL, U6 93LCxxBxxOT, X1 SG-8101CE 100Mhz, Y1 12Mhz/18pf

Commit message: starting to populate parts
Parts:
- 1V2_1, 3V3_1, 5V_1: 'LCSC Part # (none) -> C2286
- C1, C10, C12, C14, C15, C17, C20, C22, C24, C25, C26, C27, C28, C29, C3, C30, C31, C33, C34, C35, C36, C37, C38, C4, C40, C41, C5, C6, C7, C8: 'LCSC Part # (none) -> C1525
- C11, C13, C16, C18, C19, C2, C21, C23, C32, C39, C9: 'LCSC Part # (none) -> C59461
- C42, C43: 'LCSC Part # (none) -> C1555
- CDONE1: 'LCSC Part # (none) -> C434423
- D1: value 1N4448WSF-7 -> 1N4148WSF-7; 'LCSC Part # (none) -> C119617
- FB1, FB2, FB3: 'LCSC Part # (none) -> C1002
- J2: 'LCSC Part # (none) -> C160404
- J3: value FX18-120S-0.8SV20 -> FX18-120S-0.8SH; 'LCSC Part # (none) -> C598059
- USB1: 'LCSC Part # (none) -> GT-USB-7004
Changed lines of the file:
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@@
 			)
 		)
-		(property "'LCSC Part #" ""
+		(property "'LCSC Part #" "C1525"
 			(at 143.51 134.62 0)
 			(effects
@@
 			)
 		)
-		(property "'LCSC Part #" ""
+		(property "'LCSC Part #" "C59461"
 			(at 201.93 74.93 0)
 			(effects
@@
 			)
 		)
-		(property "'LCSC Part #" ""
+		(property "'LCSC Part #" "C1525"
 			(at 162.56 86.36 0)
 			(effects
@@
 			)
 		)
-		(property "'LCSC Part #" ""
+		(property "'LCSC Part #" "C160404"
 			(at 181.61 22.86 0)
 			(effects
@@
 			)
 		)
-		(property "'LCSC Part #" ""
+		(property "'LCSC Part #" "C1525"
 			(at 153.67 134.62 0)
 			(effects
@@
 			)
 		)
-		(property "'LCSC Part #" ""
+		(property "'LCSC Part #" "C1525"
 			(at 133.35 134.62 0)
 			(effects
@@
 			)
 		)
-		(property "'LCSC Part #" ""
+		(property "'LCSC Part #" "C1525"
 			(at 298.45 33.02 0)
 			(effects
@@
 			)
 		)
-		(property "'LCSC Part #" ""
+		(property "'LCSC Part #" "C1525"
 			(at 205.74 110.49 0)
 			(effects
@@
 			)
 		)
-		(property "'LCSC Part #" ""
+		(property "'LCSC Part #" "C2286"
 			(at 74.93 46.99 0)
 			(effects
@@
 			)
 		)
-		(property "Value" "FX18-120S-0.8SV20"
+		(property "Value" "FX18-120S-0.8SH"
 			(at 226.314 260.858 0)
 			(effects
@@
 			)
 		)
-		(property "'LCSC Part #" ""
+		(property "'LCSC Part #" "C598059"
 			(at 237.49 147.32 0)
 			(effects
@@
 			)
 		)
-		(property "'LCSC Part #" ""
+		(property "'LCSC Part #" "C1525"
 			(at 321.31 58.42 0)
 			(effects
@@
 			)
 		)
-		(property "'LCSC Part #" ""
+		(property "'LCSC Part #" "C1525"
 			(at 318.77 33.02 0)
 			(effects
@@
 			)
 		)
-		(property "'LCSC Part #" ""
+		(property "'LCSC Part #" "C1525"
 			(at 309.88 33.02 0)
 			(effects
@@
 			)
 		)
-		(property "'LCSC Part #" ""
+		(property "'LCSC Part #" "C1525"
 			(at 29.21 208.28 0)
 			(effects
@@
 			)
 		)
-		(property "'LCSC Part #" ""
+		(property "'LCSC Part #" "C1525"
 			(at 342.9 120.65 0)
 			(effects
@@
 			)
 		)
-		(property "'LCSC Part #" ""
+		(property "'LCSC Part #" "C59461"
 			(at 288.29 33.02 0)
 			(effects
@@
 			)
 		)
-		(property "Value" "FX18-120S-0.8SV20"
+		(property "Value" "FX18-120S-0.8SH"
 			(at 200.406 260.858 0)
 			(effects
@@
 			)
 		)
-		(property "'LCSC Part #" ""
+		(property "'LCSC Part #" "C598059"
 			(at 212.09 147.32 0)
 			(effects
@@
 			)
 		)
-		(property "'LCSC Part #" ""
+		(property "'LCSC Part #" "GT-USB-7004"
 			(at 35.56 53.34 0)
 			(effects
@@
 			)
 		)
-		(property "'LCSC Part #" ""
+		(property "'LCSC Part #" "C59461"
 			(at 90.17 114.3 0)
 			(effects
@@
 			)
 		)
-		(property "'LCSC Part #" ""
+		(property "'LCSC Part #" "C1525"
 			(at 383.54 120.65 0)
 			(effects
@@
 			)
 		)
-		(property "'LCSC Part #" ""
+		(property "'LCSC Part #" "C1525"
 			(at 363.22 120.65 0)
 			(effects
@@
 			)
 		)
-		(property "'LCSC Part #" ""
+		(property "'LCSC Part #" "C59461"
 			(at 172.72 86.36 0)
 			(effects
@@
 			)
 		)
-		(property "'LCSC Part #" ""
+		(property "'LCSC Part #" "C59461"
 			(at 54.61 171.45 0)
 			(effects
@@
 			)
 		)
-		(property "'LCSC Part #" ""
+		(property "'LCSC Part #" "C1002"
 			(at 60.96 38.1 0)
 			(effects
@@
 			)
 		)
-		(property "Value" "1N4448WSF-7"
+		(property "Value" "1N4148WSF-7"
 			(at 353.568 32.766 90)
 			(effects
@@
 			)
 		)
-		(property "'LCSC Part #" ""
+		(property "'LCSC Part #" "C119617"
 			(at 351.79 31.75 0)
 			(effects
@@
 			)
 		)
-		(property "'LCSC Part #" ""
+		(property "'LCSC Part #" "C1525"
 			(at 353.06 120.65 0)
 			(effects
@@
 			)
 		)
-		(property "'LCSC Part #" ""
+		(property "'LCSC Part #" "C1525"
 			(at 234.95 30.48 0)
 			(effects
@@
 			)
 		)
-		(property "'LCSC Part #" ""
+		(property "'LCSC Part #" "C1525"
 			(at 373.38 120.65 0)
 			(effects
@@
 			)
 		)
-		(property "'LCSC Part #" ""
+		(property "'LCSC Part #" "C59461"
 			(at 264.16 78.74 0)
 			(effects
@@
 			)
 		)
-		(property "'LCSC Part #" ""
+		(property "'LCSC Part #" "C1002"
 			(at 80.01 110.49 0)
 			(effects
@@
 			)
 		)
-		(property "'LCSC Part #" ""
+		(property "'LCSC Part #" "C59461"
 			(at 384.81 44.45 0)
 			(effects
@@
 			)
 		)
-		(property "'LCSC Part #" ""
+		(property "'LCSC Part #" "C59461"
 			(at 90.17 132.08 0)
 			(effects
@@
 			)
 		)
-		(property "'LCSC Part #" ""
+		(property "'LCSC Part #" "C1525"
 			(at 374.65 44.45 0)
 			(effects
@@
 			)
 		)
-		(property "'LCSC Part #" ""
+		(property "'LCSC Part #" "C1525"
 			(at 354.33 44.45 0)
 			(effects
@@
 			)
 		)
-		(property "'LCSC Part #" ""
+		(property "'LCSC Part #" "C1525"
 			(at 73.66 146.05 0)
 			(effects
@@
 			)
 		)
-		(property "'LCSC Part #" ""
+		(property "'LCSC Part #" "C1525"
 			(at 394.97 120.65 0)
 			(effects
@@
 			)
 		)
-		(property "'LCSC Part #" ""
+		(property "'LCSC Part #" "C1525"
 			(at 64.77 171.45 0)
 			(effects
@@
 			)
 		)
-		(property "'LCSC Part #" ""
+		(property "'LCSC Part #" "C1525"
 			(at 163.83 134.62 0)
 			(effects
@@
 			)
 		)
-		(property "'LCSC Part #" ""
+		(property "'LCSC Part #" "C59461"
 			(at 264.16 114.3 0)
 			(effects
@@
 			)
 		)
-		(property "'LCSC Part #" ""
+		(property "'LCSC Part #" "C434423"
 			(at 367.03 81.28 0)
 			(effects
@@
 			)
 		)
-		(property "'LCSC Part #" ""
+		(property "'LCSC Part #" "C2286"
 			(at 276.86 80.01 0)
 			(effects
@@
 			)
 		)
-		(property "'LCSC Part #" ""
+		(property "'LCSC Part #" "C59461"
 			(at 201.93 110.49 0)
 			(effects
@@
 			)
 		)
-		(property "'LCSC Part #" ""
+		(property "'LCSC Part #" "C2286"
 			(at 276.86 115.57 0)
 			(effects
@@
 			)
 		)
-		(property "'LCSC Part #" ""
+		(property "'LCSC Part #" "C1525"
 			(at 332.74 120.65 0)
 			(effects
@@
 			)
 		)
-		(property "'LCSC Part #" ""
+		(property "'LCSC Part #" "C1525"
 			(at 205.74 74.93 0)
 			(effects
@@
 			)
 		)
-		(property "'LCSC Part #" ""
+		(property "'LCSC Part #" "C1525"
 			(at 397.51 44.45 0)
 			(effects
@@
 			)
 		)
-		(property "'LCSC Part #" ""
+		(property "'LCSC Part #" "C1525"
 			(at 31.75 78.74 0)
 			(effects
@@
 			)
 		)
-		(property "'LCSC Part #" ""
+		(property "'LCSC Part #" "C59461"
 			(at 407.67 44.45 0)
 			(effects
@@
 			)
 		)
-		(property "'LCSC Part #" ""
+		(property "'LCSC Part #" "C1525"
 			(at 330.2 33.02 0)
 			(effects
@@
 			)
 		)
-		(property "'LCSC Part #" ""
+		(property "'LCSC Part #" "C1555"
 			(at 69.85 241.3 0)
 			(effects
@@
 			)
 		)
-		(property "'LCSC Part #" ""
+		(property "'LCSC Part #" "C1002"
 			(at 80.01 128.27 0)
 			(effects
@@
 			)
 		)
-		(property "Value" "FX18-120S-0.8SV20"
+		(property "Value" "FX18-120S-0.8SH"
 			(at 252.476 261.112 0)
 			(effects
@@
 			)
 		)
-		(property "'LCSC Part #" ""
+		(property "'LCSC Part #" "C598059"
 			(at 264.16 147.32 0)
 			(effects
@@
 			)
 		)
-		(property "'LCSC Part #" ""
+		(property "'LCSC Part #" "C1555"
 			(at 69.85 231.14 0)
 			(effects
@@
 			)
 		)
-		(property "'LCSC Part #" ""
+		(property "'LCSC Part #" "C1525"
 			(at 100.33 132.08 0)
 			(effects
@@
 			)
 		)
-		(property "'LCSC Part #" ""
+		(property "'LCSC Part #" "C1525"
 			(at 405.13 120.65 0)
 			(effects
@@
 			)
 		)
-		(property "'LCSC Part #" ""
+		(property "'LCSC Part #" "C1525"
 			(at 100.33 114.3 0)
 			(effects

Commit message: part numbers added
Parts:
- 1V2_1, 3V3_1, 5V_1: 'LCSC Part # C2286 -> (none); LCSC Part # (none) -> C2286
- C1, C10, C12, C14, C15, C17, C20, C22, C24, C25, C26, C27, C28, C29, C3, C30, C31, C33, C34, C35, C36, C37, C38, C4, C40, C41, C5, C6, C7, C8: 'LCSC Part # C1525 -> (none); LCSC Part # (none) -> C1525
- C11, C13, C16, C18, C19, C2, C21, C23, C32, C39, C9: 'LCSC Part # C59461 -> (none); LCSC Part # (none) -> C59461
- C42, C43: 'LCSC Part # C1555 -> (none); LCSC Part # (none) -> C1555
- CDONE1: 'LCSC Part # C434423 -> (none); LCSC Part # (none) -> C434423
- D1: 'LCSC Part # C119617 -> (none); LCSC Part # (none) -> C119617
- FB1, FB2, FB3: 'LCSC Part # C1002 -> (none); LCSC Part # (none) -> C1002
- J2: 'LCSC Part # C160404 -> (none); LCSC Part # (none) -> C160404
- J3: 'LCSC Part # C598059 -> (none); LCSC Part # (none) -> C598059
- L1, L2: LCSC Part # (none) -> C391305
- R1, R10, R11, R2, R21, R31, R37, R6: LCSC Part # (none) -> C4190
- R12: LCSC Part # (none) -> C23058
- R13, R15, R16, R17, R18, R19, R20, R22, R23, R34, R35, R36, R9: LCSC Part # (none) -> C25804
- R14: LCSC Part # (none) -> C7250
- R24, R25, R26, R27, R28, R29, R3, R32, R33: LCSC Part # (none) -> C21189
- R30: LCSC Part # (none) -> C22790
- R4, R5: LCSC Part # (none) -> C22775
- R7, R8: LCSC Part # (none) -> C23186
- RESET1: LCSC Part # (none) -> C221897
- U1, U4: LCSC Part # (none) -> C19188399
- U2: LCSC Part # (none) -> C1521989
- U3: LCSC Part # (none) -> C19617
- U5: LCSC Part # (none) -> C27882
- U6: LCSC Part # (none) -> C190271
- USB1: 'LCSC Part # GT-USB-7004 -> (none); LCSC Part # (none) -> GT-USB-7004
- USR1, USR2: LCSC Part # (none) -> C965807
- X1: LCSC Part # (none) -> C390559
- Y1: LCSC Part # (none) -> C390764
