File: pcb/vanillaice40/vanillaice40.kicad_sch (KiCad schematic)
At the start: 109 parts, among them J1 Conn_01x02_Pin, J2 SM04B-SRSS-TBLFSN, J3 FX18-120S-0.8SH, J4 Conn_01x06_Pin, J5 Conn_01x02_Pin, J6 Conn_01x02_Pin, J7 Conn_01x02_Pin, U1 TPS563252DRLR, U2 ICE40HX4K-TQ144, U3 W25X40CLSN, U4 TPS563252DRLR, U5 FT2232HL, U6 93LCxxBxxOT, X1 SG-8101CE 100Mhz, Y1 12Mhz/18pf

Commit message: fixed usb part #
Parts:
- USB1: LCSC Part # GT-USB-7004 -> C2686968
Changed lines of the file:
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@@
 			)
 		)
-		(property "LCSC Part #" "GT-USB-7004"
+		(property "LCSC Part #" "C2686968"
 			(at 35.56 53.34 0)
 			(effects

Commit message: pcb -> schematic footprint update
Parts:
- J2: footprint CONN_SM04B_JST -> SM04B-SRSS-TB-LF-SN:CONN_SM04B_JST
- J3: footprint CONN_120S-0.8SV20 -> FX18-120S-0-8SV20:CONN_120S-0.8SV20
- U1, U4: footprint SOT6_DRL_TEX -> PS563252DRLR:SOT6_DRL_TEX
Changed lines of the file:
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@@
 			)
 		)
+		(property "'LCSC Part #" ""
+			(at 0 345.44 0)
+			(effects
+				(font
+					(size 1.27 1.27)
+				)
+				(hide yes)
+			)
+		)
 		(pin "1"
 		)
@@
 			)
 		)
+		(property "'LCSC Part #" ""
+			(at 0 45.72 0)
+			(effects
+				(font
+					(size 1.27 1.27)
+				)
+				(hide yes)
+			)
+		)
 		(pin "1"
 		)
@@
 			)
 		)
-		(property "Footprint" "CONN_SM04B_JST"
+		(property "Footprint" "SM04B-SRSS-TB-LF-SN:CONN_SM04B_JST"
 			(at 181.61 22.86 0)
 			(effects
@@
 			)
 		)
+		(property "'LCSC Part #" ""
+			(at 0 287.02 0)
+			(effects
+				(font
+					(size 1.27 1.27)
+				)
+				(hide yes)
+			)
+		)
 		(pin "5"
 		)
@@
 			)
 		)
-		(property "Footprint" "CONN_120S-0.8SV20"
+		(property "Footprint" "FX18-120S-0-8SV20:CONN_120S-0.8SV20"
 			(at 237.49 147.32 0)
 			(effects
@@
 			)
 		)
-		(property "Footprint" "CONN_120S-0.8SV20"
+		(property "Footprint" "FX18-120S-0-8SV20:CONN_120S-0.8SV20"
 			(at 212.09 147.32 0)
 			(effects
@@
 			)
 		)
+		(property "'LCSC Part #" ""
+			(at 0 111.76 0)
+			(effects
+				(font
+					(size 1.27 1.27)
+				)
+				(hide yes)
+			)
+		)
 		(pin "1"
 		)
@@
 			)
 		)
-		(property "Footprint" "SOT6_DRL_TEX"
+		(property "Footprint" "PS563252DRLR:SOT6_DRL_TEX"
 			(at 208.28 106.68 0)
 			(effects
@@
 			)
 		)
-		(property "Footprint" "SOT6_DRL_TEX"
+		(property "Footprint" "PS563252DRLR:SOT6_DRL_TEX"
 			(at 208.28 71.12 0)
 			(effects
@@
 			)
 		)
+		(property "'LCSC Part #" ""
+			(at 0 162.56 0)
+			(effects
+				(font
+					(size 1.27 1.27)
+				)
+				(hide yes)
+			)
+		)
 		(pin "1"
 		)
@@
 			)
 		)
-		(property "Footprint" "CONN_120S-0.8SV20"
+		(property "Footprint" "FX18-120S-0-8SV20:CONN_120S-0.8SV20"
 			(at 264.16 147.32 0)
 			(effects

Commit message: custom fx18 footprint
Parts:
- J3: footprint FX18-120S-0-8SV20:CONN_120S-0.8SV20 -> custom:CUSTOM_FX_120S-0.8SH20
Changed lines of the file:
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@@
 			)
 		)
-		(property "Footprint" "FX18-120S-0-8SV20:CONN_120S-0.8SV20"
+		(property "Footprint" "custom:CUSTOM_FX_120S-0.8SH20"
 			(at 237.49 147.32 0)
 			(effects
@@
 			)
 		)
-		(property "Footprint" "FX18-120S-0-8SV20:CONN_120S-0.8SV20"
+		(property "Footprint" "custom:CUSTOM_FX_120S-0.8SH20"
 			(at 212.09 147.32 0)
 			(effects
@@
 			)
 		)
-		(property "Footprint" "FX18-120S-0-8SV20:CONN_120S-0.8SV20"
+		(property "Footprint" "custom:CUSTOM_FX_120S-0.8SH20"
 			(at 264.16 147.32 0)
 			(effects

Commit message: start of jclpcb pos fixes
Parts:
- USB1: JLCPCB Position Offset (none) -> 0,1.3335
Changed lines of the file:
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@@
+			)
+		)
+		(property "JLCPCB Position Offset" "0,1.3335"
+			(at 35.56 53.34 0)
+			(effects
+				(font
+					(size 1.27 1.27)
+				)
+				(hide yes)
 			)
 		)

Commit message: all parts jlcpcb pos/rotated
Parts:
- J2: JLCPCB Position Offset (none) -> 1.524,-2.032
- U1, U4: JLCPCB Rotation Offset (none) -> -90
- U5: JLCPCB Rotation Offset (none) -> 90

Commit message: digikey part numbers
Parts:
- 1V2_1, 3V3_1, 5V_1: Digi-Key Part Number (none) -> 732-4978-1-ND
- C1, C10, C12, C14, C15, C17, C20, C22, C24, C25, C26, C27, C28, C29, C3, C30, C31, C33, C34, C35, C36, C37, C38, C4, C40, C41, C5, C6, C7, C8: Digi-Key Part Number (none) -> 490-6328-1-ND
- C11, C13, C16, C18, C19, C2, C21, C23, C32, C39, C9: Digi-Key Part Number (none) -> 490-7611-1-ND
- C42, C43: Digi-Key Part Number (none) -> 490-5869-1-ND
- CDONE1: Digi-Key Part Number (none) -> 732-4971-1-ND
- D1: Digi-Key Part Number (none) -> 1N4148WSF-7DICT-ND
- FB1, FB2, FB3: Digi-Key Part Number (none) -> 490-5258-1-ND
- J2: Digi-Key Part Number (none) -> 455-SM04B-SRSS-TBCT-ND
- J3: Digi-Key Part Number (none) -> FX18-120S-0.8SH
- L1, L2: Digi-Key Part Number (none) -> 490-10649-1-ND
- R1, R10, R11, R2, R21, R31, R37, R6: Digi-Key Part Number (none) -> 118-CR0603-FX-2201ELFCT-ND
- R12: Digi-Key Part Number (none) -> CR0603-FX-4532ELFCT-ND
- R13, R15, R16, R17, R18, R19, R20, R22, R23, R34, R35, R36, R9: Digi-Key Part Number (none) -> CR0603-FX-1002ELFCT-ND
- R14: Digi-Key Part Number (none) -> CR0603-FW-1005ELFCT-ND
- R24, R25, R26, R27, R28, R29, R3, R32, R33: Digi-Key Part Number (none) -> CR0603-J/-000ELFCT-ND
- R30: Digi-Key Part Number (none) -> 118-CR0603-FX-1202ELFCT-ND
- R4, R5: Digi-Key Part Number (none) -> CR0603-FX-1000ELFCT-ND
- R7, R8: Digi-Key Part Number (none) -> CR0603-FX-5101ELFCT-ND
- RESET1: Digi-Key Part Number (none) -> CKN10503CT-ND
- U1, U4: Digi-Key Part Number (none) -> 296-TPS563252DRLRCT-ND
- U2: Digi-Key Part Number (none) -> ICE40HX4K-TQ144
- U3: Digi-Key Part Number (none) -> W25X40CLSNIG-ND
- U5: Digi-Key Part Number (none) -> 768-1024-1-ND
- U6: Digi-Key Part Number (none) -> 93LC56BT-I/OTCT-ND
- USB1: Digi-Key Part Number (none) -> 2073-USB4105-GF-ACT-ND
- USR1, USR2: Digi-Key Part Number (none) -> 732-4966-1-ND
- X1: Digi-Key Part Number (none) -> 50-ECS-3225MVQ-1000-CN-CT-ND
- Y1: Digi-Key Part Number (none) -> 535-10261-1-ND
