File: pcb/breakout-pmod/breakout-pmod.kicad_pcb (KiCad board)
At the start: 4 copper layers, 88.9 x 100 mm, 13 parts, among them J1 FX18-120P-0.8SV20

Commit message: [pmod] fix order of AB pmod
Connections:
- J1 pad 4: /AB_02 -> /AB_05
- J1 pad 5: /AB_03 -> /AB_02
- J1 pad 6: /AB_04 -> /AB_06
- J1 pad 7: /AB_05 -> /AB_03
- J1 pad 8: /AB_06 -> /AB_07
- J1 pad 9: /AB_07 -> /AB_04
- PM1 pad 2: /AB_03 -> /AB_02
- PM1 pad 3: /AB_05 -> /AB_03
- PM1 pad 4: /AB_07 -> /AB_04
- PM1 pad 7: /AB_02 -> /AB_05
- PM1 pad 8: /AB_04 -> /AB_06
- PM1 pad 9: /AB_06 -> /AB_07
Routing:
- net /AB_02: track 23.3 -> 20.9 mm
- net /AB_07: track 25.3 -> 27.7 mm
- net /AB_06: track 27.7 -> 25.4 mm
- net /AB_03: track 20.9 -> 23.1 mm
