File: pcb/breakout-pmod/breakout-pmod.kicad_pcb (KiCad board)
At the start: 4 copper layers, 88.9 x 100 mm, 13 parts, among them J1 FX18-120P-0.8SV20

Commit message: [pmod] fix order of KL pmod
Connections:
- J1 pad 52: /KL_02 -> /KL_05
- J1 pad 53: /KL_03 -> /KL_02
- J1 pad 54: /KL_04 -> /KL_06
- J1 pad 55: /KL_05 -> /KL_03
- J1 pad 56: /KL_06 -> /KL_07
- J1 pad 57: /KL_07 -> /KL_04
- PM7 pad 2: /KL_03 -> /KL_02
- PM7 pad 3: /KL_05 -> /KL_03
- PM7 pad 4: /KL_07 -> /KL_04
- PM7 pad 7: /KL_02 -> /KL_05
- PM7 pad 8: /KL_04 -> /KL_06
- PM7 pad 9: /KL_06 -> /KL_07
Routing:
- net /KL_04: track 69.9 -> 61.3 mm
- net /KL_05: track 65.2 -> 73.1 mm
- net /KL_07: track 61.3 -> 66.3 mm
- net /KL_02: track 73.1 -> 68.4 mm
- net /KL_06: track 66.3 -> 69.9 mm
- net /KL_03: track 68.4 -> 65.2 mm
Changed lines of the file:
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@@
 			(layers "*.Cu" "*.Mask")
 			(remove_unused_layers no)
-			(net 34 "/KL_03")
+			(net 14 "/KL_02")
 			(pinfunction "Pin_2")
 			(pintype "passive")
@@
 			(layers "*.Cu" "*.Mask")
 			(remove_unused_layers no)
-			(net 9 "/KL_05")
+			(net 34 "/KL_03")
 			(pinfunction "Pin_3")
 			(pintype "passive")
@@
 			(layers "*.Cu" "*.Mask")
 			(remove_unused_layers no)
-			(net 70 "/KL_07")
+			(net 94 "/KL_04")
 			(pinfunction "Pin_4")
 			(pintype "passive")
@@
 			(layers "*.Cu" "*.Mask")
 			(remove_unused_layers no)
-			(net 14 "/KL_02")
+			(net 9 "/KL_05")
 			(pinfunction "Pin_7")
 			(pintype "passive")
@@
 			(layers "*.Cu" "*.Mask")
 			(remove_unused_layers no)
-			(net 94 "/KL_04")
+			(net 30 "/KL_06")
 			(pinfunction "Pin_8")
 			(pintype "passive")
@@
 			(layers "*.Cu" "*.Mask")
 			(remove_unused_layers no)
-			(net 30 "/KL_06")
+			(net 70 "/KL_07")
 			(pinfunction "Pin_9")
 			(pintype "passive")
@@
 			(size 0.4572 2.2098)
 			(layers "F.Cu" "F.Paste" "F.Mask")
-			(net 14 "/KL_02")
+			(net 9 "/KL_05")
 			(pinfunction "52")
 			(pintype "passive")
@@
 			(size 0.4572 2.2098)
 			(layers "F.Cu" "F.Paste" "F.Mask")
-			(net 34 "/KL_03")
+			(net 14 "/KL_02")
 			(pinfunction "53")
 			(pintype "passive")
@@
 			(size 0.4572 2.2098)
 			(layers "F.Cu" "F.Paste" "F.Mask")
-			(net 94 "/KL_04")
+			(net 30 "/KL_06")
 			(pinfunction "54")
 			(pintype "passive")
@@
 			(size 0.4572 2.2098)
 			(layers "F.Cu" "F.Paste" "F.Mask")
-			(net 9 "/KL_05")
+			(net 34 "/KL_03")
 			(pinfunction "55")
 			(pintype "passive")
@@
 			(size 0.4572 2.2098)
 			(layers "F.Cu" "F.Paste" "F.Mask")
-			(net 30 "/KL_06")
+			(net 70 "/KL_07")
 			(pinfunction "56")
 			(pintype "passive")
@@
 			(size 0.4572 2.2098)
 			(layers "F.Cu" "F.Paste" "F.Mask")
-			(net 70 "/KL_07")
+			(net 94 "/KL_04")
 			(pinfunction "57")
 			(pintype "passive")
@@
 		)
 	)
-	(gr_text "02/08"
-		(at 105.156 126.365 90)
-		(layer "F.SilkS")
-		(effects
-			(font
-				(size 0.7 0.7)
-				(thickness 0.15)
-				(bold yes)
-			)
-			(justify left bottom)
-		)
-	)
 	(gr_text "3V3"
 		(at 114.935 86.614 0)
@@
 		)
 	)
-	(gr_text "06/10"
-		(at 100.076 126.365 90)
+	(gr_text "06/02"
+		(at 105.2 126.365 90)
 		(layer "F.SilkS")
 		(effects
@@
 		)
 	)
-	(gr_text "05/09"
-		(at 102.616 126.365 90)
+	(gr_text "05/01"
+		(at 107.74 126.365 90)
 		(layer "F.SilkS")
 		(effects
@@
 	)
 	(gr_text "05/01"
-		(at 130.683 124.968 90)
+		(at 130.57 124.95 90)
 		(layer "F.SilkS")
 		(effects
@@
 	)
 	(gr_text "08/04"
-		(at 123.063 124.968 90)
+		(at 122.95 124.95 90)
 		(layer "F.SilkS")
 		(effects
@@
 	)
 	(gr_text "07/03"
-		(at 125.603 124.968 90)
+		(at 125.49 124.95 90)
 		(layer "F.SilkS")
 		(effects
@@
 		)
 	)
-	(gr_text "01/07"
-		(at 107.696 126.365 90)
-		(layer "F.SilkS")
-		(effects
-			(font
-				(size 0.7 0.7)
-				(thickness 0.15)
-				(bold yes)
-			)
-			(justify left bottom)
-		)
-	)
 	(gr_text "3V3"
 		(at 94.996 126.365 90)
@@
 		)
 	)
+	(gr_text "07/03"
+		(at 102.66 126.365 90)
+		(layer "F.SilkS")
+		(effects
+			(font
+				(size 0.7 0.7)
+				(thickness 0.15)
+				(bold yes)
+			)
+			(justify left bottom)
+		)
+	)
 	(gr_text "03/07"
 		(at 54.41 60.452 90)
@@
 	)
 	(gr_text "06/02"
-		(at 128.143 124.968 90)
+		(at 128.03 124.95 90)
 		(layer "F.SilkS")
 		(effects
@@
 		)
 	)
+	(gr_text "08/04"
+		(at 100.12 126.365 90)
+		(layer "F.SilkS")
+		(effects
+			(font
+				(size 0.7 0.7)
+				(thickness 0.15)
+				(bold yes)
+			)
+			(justify left bottom)
+		)
+	)
 	(segment
 		(start 53.150999 104.529996)
@@
 	)
 	(segment
-		(start 101.531996 110.929996)
-		(end 102.2 111.598)
+		(start 102.941996 108.529996)
+		(end 106.02 111.608)
 		(width 0.156464)
 		(layer "F.Cu")
@@
 	)
 	(segment
-		(start 53.150999 110.929996)
-		(end 101.531996 110.929996)
+		(start 106.02 128.755)
+		(end 107.28 130.015)
 		(width 0.156464)
 		(layer "F.Cu")
@@
 	)
 	(segment
-		(start 102.2 111.598)
-		(end 102.2 127.475)
+		(start 106.02 111.608)
+		(end 106.02 128.755)
+		(width 0.156464)
+		(layer "F.Cu")
+		(net 9)
+	)
+	(segment
+		(start 53.150999 108.529996)
+		(end 102.941996 108.529996)
 		(width 0.156464)
 		(layer "F.Cu")
@@
 	)
 	(segment
-		(start 102.941996 108.529996)
-		(end 106.02 111.608)
-		(width 0.156464)
-		(layer "F.Cu")
-		(net 14)
-	)
-	(segment
-		(start 106.02 128.755)
-		(end 107.28 130.015)
+		(start 102.471997 109.329997)
+		(end 104.74 111.598)
 		(width 0.156464)
 		(layer "F.Cu")
@@
 	)
 	(segment
-		(start 106.02 111.608)
-		(end 106.02 128.755)
+		(start 104.74 111.598)
+		(end 104.74 127.475)
 		(width 0.156464)
 		(layer "F.Cu")
@@
 	)
 	(segment
-		(start 53.150999 108.529996)
-		(end 102.941996 108.529996)
+		(start 53.150999 109.329997)
+		(end 102.471997 109.329997)
 		(width 0.156464)
 		(layer "F.Cu")
@@
 	)
 	(segment
-		(start 100.92 112.13)
-		(end 100.92 128.735)
+		(start 53.150999 110.129998)
+		(end 102.001998 110.129998)
 		(width 0.156464)
 		(layer "F.Cu")
@@
 	)
 	(segment
-		(start 100.92 128.735)
-		(end 102.2 130.015)
+		(start 103.49 111.618)
+		(end 103.49 128.765)
 		(width 0.156464)
 		(layer "F.Cu")
@@
 	)
 	(segment
-		(start 100.519997 111.729997)
-		(end 100.92 112.13)
+		(start 103.49 128.765)
+		(end 104.74 130.015)
 		(width 0.156464)
 		(layer "F.Cu")
@@
 	)
 	(segment
-		(start 53.150999 111.729997)
-		(end 100.519997 111.729997)
+		(start 102.001998 110.129998)
+		(end 103.49 111.618)
 		(width 0.156464)
 		(layer "F.Cu")
@@
 	)
 	(segment
-		(start 102.471997 109.329997)
-		(end 104.74 111.598)
+		(start 101.531996 110.929996)
+		(end 102.2 111.598)
 		(width 0.156464)
 		(layer "F.Cu")
@@
 	)
 	(segment
-		(start 104.74 111.598)
-		(end 104.74 127.475)
+		(start 53.150999 110.929996)
+		(end 101.531996 110.929996)
 		(width 0.156464)
 		(layer "F.Cu")
@@
 	)
 	(segment
-		(start 53.150999 109.329997)
-		(end 102.471997 109.329997)
+		(start 102.2 111.598)
+		(end 102.2 127.475)
 		(width 0.156464)
 		(layer "F.Cu")
@@
 	)
 	(segment
-		(start 53.150999 112.529996)
-		(end 99.321996 112.529996)
+		(start 100.92 112.13)
+		(end 100.92 128.735)
 		(width 0.156464)
 		(layer "F.Cu")
@@
 	)
 	(segment
-		(start 99.321996 112.529996)
-		(end 99.66 112.868)
+		(start 100.92 128.735)
+		(end 102.2 130.015)
 		(width 0.156464)
 		(layer "F.Cu")
@@
 	)
 	(segment
-		(start 99.66 112.868)
-		(end 99.66 127.475)
+		(start 100.519997 111.729997)
+		(end 100.92 112.13)
+		(width 0.156464)
+		(layer "F.Cu")
+		(net 70)
+	)
+	(segment
+		(start 53.150999 111.729997)
+		(end 100.519997 111.729997)
 		(width 0.156464)
 		(layer "F.Cu")
@@
 	)
 	(segment
-		(start 53.150999 110.129998)
-		(end 102.001998 110.129998)
-		(width 0.156464)
-		(layer "F.Cu")
-		(net 94)
-	)
-	(segment
-		(start 103.49 111.618)
-		(end 103.49 128.765)
+		(start 53.150999 112.529996)
+		(end 99.321996 112.529996)
 		(width 0.156464)
 		(layer "F.Cu")
@@
 	)
 	(segment
-		(start 103.49 128.765)
-		(end 104.74 130.015)
+		(start 99.321996 112.529996)
+		(end 99.66 112.868)
 		(width 0.156464)
 		(layer "F.Cu")
@@
 	)
 	(segment
-		(start 102.001998 110.129998)
-		(end 103.49 111.618)
+		(start 99.66 112.868)
+		(end 99.66 127.475)
 		(width 0.156464)
 		(layer "F.Cu")

Commit message: [pmod] fix order of HG pmod
Connections:
- J1 pad 92: /HG_02 -> /HG_05
- J1 pad 93: /HG_03 -> /HG_02
- J1 pad 94: /HG_04 -> /HG_06
- J1 pad 95: /HG_05 -> /HG_03
- J1 pad 96: /HG_06 -> /HG_07
- J1 pad 97: /HG_07 -> /HG_04
- PM6 pad 2: /HG_03 -> /HG_02
- PM6 pad 3: /HG_05 -> /HG_03
- PM6 pad 4: /HG_07 -> /HG_04
- PM6 pad 7: /HG_02 -> /HG_05
- PM6 pad 8: /HG_04 -> /HG_06
- PM6 pad 9: /HG_06 -> /HG_07
Routing:
- net /HG_04: track 62.2 -> 53.7 mm
- net /HG_05: track 57.5 -> 65.4 mm
- net /HG_07: track 53.7 -> 58.9 mm
- net /HG_02: track 65.4 -> 60.7 mm
- net /HG_06: track 58.9 -> 62.2 mm
- net /HG_03: track 60.7 -> 57.5 mm

Commit message: [pmod] fix order of LK pmod
Connections:
- J1 pad 112: /LK_02 -> /LK_05
- J1 pad 113: /LK_03 -> /LK_02
- J1 pad 114: /LK_04 -> /LK_06
- J1 pad 115: /LK_05 -> /LK_03
- J1 pad 116: /LK_06 -> /LK_07
- J1 pad 117: /LK_07 -> /LK_04
- PM5 pad 2: /LK_03 -> /LK_02
- PM5 pad 3: /LK_05 -> /LK_03
- PM5 pad 4: /LK_07 -> /LK_04
- PM5 pad 7: /LK_02 -> /LK_05
- PM5 pad 8: /LK_04 -> /LK_06
- PM5 pad 9: /LK_06 -> /LK_07
Routing:
- net /LK_05: track 24.5 -> 31.9 mm
- net /LK_04: track 28.8 -> 21.7 mm
- net /LK_02: track 31.9 -> 27.4 mm
- net /LK_07: track 21.7 -> 26.1 mm
- net /LK_03: track 27.4 -> 24.5 mm
- net /LK_06: track 26.1 -> 28.8 mm
Other:
- board text added: "LK"

Commit message: [pmod] fix order of FE pmod
Note: this is actually wired backwards on the PCB
and probably won't mirror correctly.
Connections:
- J1 pad 83: /FE_01 -> /FE_08
- J1 pad 84: /FE_02 -> /FE_04
- J1 pad 85: /FE_03 -> /FE_07
- J1 pad 86: /FE_04 -> /FE_03
- J1 pad 87: /FE_05 -> /FE_06
- J1 pad 88: /FE_06 -> /FE_02
- J1 pad 89: /FE_07 -> /FE_05
- J1 pad 90: /FE_08 -> /FE_01
- PM10 pad 1: /FE_08 -> /FE_01
- PM10 pad 10: /FE_01 -> /FE_08
- PM10 pad 2: /FE_06 -> /FE_02
- PM10 pad 3: /FE_04 -> /FE_03
- PM10 pad 4: /FE_02 -> /FE_04
- PM10 pad 7: /FE_07 -> /FE_05
- PM10 pad 8: /FE_05 -> /FE_06
- PM10 pad 9: /FE_03 -> /FE_07
Routing:
- net /FE_08: track 60.0 -> 68.1 mm
- net /FE_01: track 68.1 -> 60.0 mm
- net /FE_07: track 58.6 -> 64.9 mm
- net /FE_02: track 69.5 -> 63.2 mm
- net /FE_05: track 61.8 -> 58.6 mm
- net /FE_04: track 66.4 -> 69.5 mm
- net /FE_03: track 64.9 -> 66.4 mm
- net /FE_06: track 63.2 -> 61.8 mm
Other:
- board text added: "JI"

Commit message: [pmod] fix order of JI pmod
Connections:
- J1 pad 101: /JI_01 -> /JI_08
- J1 pad 102: /JI_02 -> /JI_04
- J1 pad 103: /JI_03 -> /JI_07
- J1 pad 104: /JI_04 -> /JI_03
- J1 pad 105: /JI_05 -> /JI_06
- J1 pad 106: /JI_06 -> /JI_02
- J1 pad 107: /JI_07 -> /JI_05
- J1 pad 108: /JI_08 -> /JI_01
- PM9 pad 1: /JI_08 -> /JI_01
- PM9 pad 10: /JI_01 -> /JI_08
- PM9 pad 2: /JI_06 -> /JI_02
- PM9 pad 3: /JI_04 -> /JI_03
- PM9 pad 4: /JI_02 -> /JI_04
- PM9 pad 7: /JI_07 -> /JI_05
- PM9 pad 8: /JI_05 -> /JI_06
- PM9 pad 9: /JI_03 -> /JI_07
Routing:
- net /JI_08: track 30.6 -> 37.7 mm
- net /JI_01: track 37.7 -> 30.6 mm
- net /JI_02: track 39.3 -> 33.5 mm
- net /JI_07: track 29.1 -> 34.8 mm
- net /JI_04: track 36.4 -> 39.3 mm
- net /JI_05: track 32.0 -> 29.1 mm
- net /JI_06: track 33.5 -> 32.0 mm
- net /JI_03: track 34.8 -> 36.4 mm
