File: pcb/breakout-tri-sram/a2d_buffers.kicad_sch (KiCad schematic)
At the start: 27 parts, among them U201 74LS573, U202 74LS573, U203 74LS573, U204 74LS573, U205 74LS573, U206 74LS573, U207 74LS573, U208 74LS573, U209 74LS573, U210 74LS573, U211 74LS573, U212 74LS573

Commit message: [pcb][tri-sram] tri-sram complete
squashed big-bus branch
Parts:
- renumbered C203 to C202, C212 to C203, C221 to C204, C230 to C205, C204 to C206, C206 to C207, C218 to C208, C227 to C209, C236 to C210, C207 to C211, C209 to C212, C215 to C213, C224 to C214, C233 to C215, U204 to U202, U207 to U203, U210 to U204, U202 to U205, U209 to U207, U212 to U208, U203 to U209, U205 to U210, U208 to U211, U211 to U212
Connections:
- net A2D_X_A1 is gone; now on net A2D_B3: U203.2 (D0), U207.2 (D0), U211.2 (D0)
- net A2D_X_A2 is gone; now on net A2D_B2: U203.3 (D1), U207.3 (D1), U211.3 (D1)
- net A2D_X_A3 is gone; now on net A2D_B1: U203.4 (D2), U207.4 (D2), U211.4 (D2)
- net A2D_X_A4 is gone; now on net A2D_B0: U203.5 (D3), U207.5 (D3), U211.5 (D3)
- net 0_A1: now also U203.12 (Q7); no longer U203.19 (Q0)
- net 0_A2: now also U203.13 (Q6); no longer U203.18 (Q1)
- net 0_A3: now also U203.14 (Q5); no longer U203.17 (Q2)
- net 0_A4: now also U203.15 (Q4); no longer U203.16 (Q3)
- net 0_D0: now also U203.16 (Q3); no longer U203.12 (Q7)
- net 0_D1: now also U203.17 (Q2); no longer U203.13 (Q6)
- net 0_D10: now also U204.17 (Q2); no longer U204.14 (Q5)
- net 0_D11: now also U204.16 (Q3); no longer U204.15 (Q4)
- net 0_D2: now also U203.18 (Q1); no longer U203.14 (Q5)
- net 0_D3: now also U203.19 (Q0); no longer U203.15 (Q4)
- net 0_D4: now also U204.12 (Q7); no longer U204.19 (Q0)
- net 0_D5: now also U204.13 (Q6); no longer U204.18 (Q1)
- net 0_D6: now also U204.14 (Q5); no longer U204.17 (Q2)
- net 0_D7: now also U204.15 (Q4); no longer U204.16 (Q3)
- net 0_D8: now also U204.19 (Q0); no longer U204.12 (Q7)
- net 0_D9: now also U204.18 (Q1); no longer U204.13 (Q6)
- net 1_A1: now also U207.12 (Q7); no longer U207.19 (Q0)
- net 1_A2: now also U207.13 (Q6); no longer U207.18 (Q1)
- net 1_A3: now also U207.14 (Q5); no longer U207.17 (Q2)
- net 1_A4: now also U207.15 (Q4); no longer U207.16 (Q3)
- net 1_D0: now also U207.16 (Q3); no longer U207.12 (Q7)
- net 1_D1: now also U207.17 (Q2); no longer U207.13 (Q6)
- net 1_D10: now also U208.17 (Q2); no longer U208.14 (Q5)
- net 1_D11: now also U208.16 (Q3); no longer U208.15 (Q4)
- net 1_D2: now also U207.18 (Q1); no longer U207.14 (Q5)
- net 1_D3: now also U207.19 (Q0); no longer U207.15 (Q4)
- net 1_D4: now also U208.12 (Q7); no longer U208.19 (Q0)
- net 1_D5: now also U208.13 (Q6); no longer U208.18 (Q1)
- net 1_D6: now also U208.14 (Q5); no longer U208.17 (Q2)
- net 1_D7: now also U208.15 (Q4); no longer U208.16 (Q3)
- net 1_D8: now also U208.19 (Q0); no longer U208.12 (Q7)
- net 1_D9: now also U208.18 (Q1); no longer U208.13 (Q6)
- net 2_A1: now also U211.12 (Q7); no longer U211.19 (Q0)
- net 2_A2: now also U211.13 (Q6); no longer U211.18 (Q1)
- net 2_A3: now also U211.14 (Q5); no longer U211.17 (Q2)
- net 2_A4: now also U211.15 (Q4); no longer U211.16 (Q3)
- net 2_D0: now also U211.16 (Q3); no longer U211.12 (Q7)
- net 2_D1: now also U211.17 (Q2); no longer U211.13 (Q6)
- net 2_D10: now also U212.17 (Q2); no longer U212.14 (Q5)
- net 2_D11: now also U212.16 (Q3); no longer U212.15 (Q4)
- net 2_D2: now also U211.18 (Q1); no longer U211.14 (Q5)
- net 2_D3: now also U211.19 (Q0); no longer U211.15 (Q4)
- net 2_D4: now also U212.12 (Q7); no longer U212.19 (Q0)
- net 2_D5: now also U212.13 (Q6); no longer U212.18 (Q1)
- net 2_D6: now also U212.14 (Q5); no longer U212.17 (Q2)
- net 2_D7: now also U212.15 (Q4); no longer U212.16 (Q3)
- net 2_D8: now also U212.19 (Q0); no longer U212.12 (Q7)
- net 2_D9: now also U212.18 (Q1); no longer U212.13 (Q6)
- net A2D_B0: no longer U203.9 (D7), U207.9 (D7), U211.9 (D7)
- net A2D_B1: no longer U203.8 (D6), U207.8 (D6), U211.8 (D6)
- net A2D_B2: no longer U203.7 (D5), U207.7 (D5), U211.7 (D5)
- net A2D_B3: no longer U203.6 (D4), U207.6 (D4), U211.6 (D4)
- net A2D_G0: now also U204.9 (D7), U208.9 (D7), U212.9 (D7); no longer U204.2 (D0), U208.2 (D0), U212.2 (D0)
- net A2D_G1: now also U204.8 (D6), U208.8 (D6), U212.8 (D6); no longer U204.3 (D1), U208.3 (D1), U212.3 (D1)
- net A2D_G2: now also U204.7 (D5), U208.7 (D5), U212.7 (D5); no longer U204.4 (D2), U208.4 (D2), U212.4 (D2)
- net A2D_G3: now also U204.6 (D4), U208.6 (D4), U212.6 (D4); no longer U204.5 (D3), U208.5 (D3), U212.5 (D3)
- net A2D_R0: now also U204.2 (D0), U208.2 (D0), U212.2 (D0); no longer U204.9 (D7), U208.9 (D7), U212.9 (D7)
- net A2D_R1: now also U204.3 (D1), U208.3 (D1), U212.3 (D1); no longer U204.8 (D6), U208.8 (D6), U212.8 (D6)
- net A2D_R2: now also U204.4 (D2), U208.4 (D2), U212.4 (D2); no longer U204.7 (D5), U208.7 (D5), U212.7 (D5)
- net A2D_R3: now also U204.5 (D3), U208.5 (D3), U212.5 (D3); no longer U204.6 (D4), U208.6 (D4), U212.6 (D4)
- net A2D_X_A0 renamed A2D_X0
- net A2D_X_A5 renamed A2D_X5
- net A2D_X_A6 renamed A2D_X6
- net A2D_X_A7 renamed A2D_X7
- net A2D_X_A8 renamed A2D_X8
- net A2D_X_A9 renamed A2D_X9
- net A2D_Y_A0 renamed A2D_Y0
- net A2D_Y_A1 renamed A2D_Y1
- net A2D_Y_A2 renamed A2D_Y2
- net A2D_Y_A3 renamed A2D_Y3
- net A2D_Y_A4 renamed A2D_Y4
- net A2D_Y_A5 renamed A2D_Y5
- net A2D_Y_A6 renamed A2D_Y6
- net A2D_Y_A7 renamed A2D_Y7
- net A2D_Y_A8 renamed A2D_Y8
- net A2D_Y_A9 renamed A2D_Y9
- new net A2D_X1: U203.9 (D7), U207.9 (D7), U211.9 (D7)
- new net A2D_X2: U203.8 (D6), U207.8 (D6), U211.8 (D6)
- new net A2D_X3: U203.7 (D5), U207.7 (D5), U211.7 (D5)
- new net A2D_X4: U203.6 (D4), U207.6 (D4), U211.6 (D4)
Other:
- moved on the sheet: C208, C209, C210, U206, U207, U208

Commit message: [pcb][tri-sram] add part numbers
Parts:
- U201, U202, U203, U204, U205, U206, U207, U208, U209, U210, U211, U212: Digi-Key Part Number (none) -> 264-74LCX541FT(AE)CT-ND
Changed lines of the file:
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@@
 			)
 		)
+		(property "Digi-Key Part Number" "264-74LCX541FT(AE)CT-ND"
+			(at 60.96 50.8 0)
+			(effects
+				(font
+					(size 1.27 1.27)
+				)
+				(hide yes)
+			)
+		)
 		(pin "5"
 		)
@@
 			)
 		)
+		(property "Digi-Key Part Number" "264-74LCX541FT(AE)CT-ND"
+			(at 60.96 111.76 0)
+			(effects
+				(font
+					(size 1.27 1.27)
+				)
+				(hide yes)
+			)
+		)
 		(pin "5"
 		)
@@
 			)
 		)
+		(property "Digi-Key Part Number" "264-74LCX541FT(AE)CT-ND"
+			(at 60.96 171.45 0)
+			(effects
+				(font
+					(size 1.27 1.27)
+				)
+				(hide yes)
+			)
+		)
 		(pin "5"
 		)
@@
 			)
 		)
+		(property "Digi-Key Part Number" "264-74LCX541FT(AE)CT-ND"
+			(at 157.48 171.45 0)
+			(effects
+				(font
+					(size 1.27 1.27)
+				)
+				(hide yes)
+			)
+		)
 		(pin "5"
 		)
@@
 			)
 		)
+		(property "Digi-Key Part Number" "264-74LCX541FT(AE)CT-ND"
+			(at 252.73 171.45 0)
+			(effects
+				(font
+					(size 1.27 1.27)
+				)
+				(hide yes)
+			)
+		)
 		(pin "5"
 		)
@@
 			)
 		)
+		(property "Digi-Key Part Number" "264-74LCX541FT(AE)CT-ND"
+			(at 60.96 234.95 0)
+			(effects
+				(font
+					(size 1.27 1.27)
+				)
+				(hide yes)
+			)
+		)
 		(pin "5"
 		)
@@
 			)
 		)
+		(property "Digi-Key Part Number" "264-74LCX541FT(AE)CT-ND"
+			(at 157.48 111.76 0)
+			(effects
+				(font
+					(size 1.27 1.27)
+				)
+				(hide yes)
+			)
+		)
 		(pin "5"
 		)
@@
 			)
 		)
+		(property "Digi-Key Part Number" "264-74LCX541FT(AE)CT-ND"
+			(at 157.48 50.8 0)
+			(effects
+				(font
+					(size 1.27 1.27)
+				)
+				(hide yes)
+			)
+		)
 		(pin "5"
 		)
@@
 			)
 		)
+		(property "Digi-Key Part Number" "264-74LCX541FT(AE)CT-ND"
+			(at 157.48 234.95 0)
+			(effects
+				(font
+					(size 1.27 1.27)
+				)
+				(hide yes)
+			)
+		)
 		(pin "5"
 		)
@@
 			)
 		)
+		(property "Digi-Key Part Number" "264-74LCX541FT(AE)CT-ND"
+			(at 252.73 50.8 0)
+			(effects
+				(font
+					(size 1.27 1.27)
+				)
+				(hide yes)
+			)
+		)
 		(pin "5"
 		)
@@
 			)
 		)
+		(property "Digi-Key Part Number" "264-74LCX541FT(AE)CT-ND"
+			(at 252.73 234.95 0)
+			(effects
+				(font
+					(size 1.27 1.27)
+				)
+				(hide yes)
+			)
+		)
 		(pin "5"
 		)
@@
 			(at 252.73 111.76 0)
 			(effects
+				(font
+					(size 1.27 1.27)
+				)
+				(hide yes)
+			)
+		)
+		(property "Digi-Key Part Number" "264-74LCX541FT(AE)CT-ND"
+			(at 252.73 111.76 0)
+			(effects
