File: pcb/breakout-tri-sram/vga_addr_buffers.kicad_sch (KiCad schematic)
At the start: 21 parts, among them U501 74LS573, U502 74LS573, U503 74LS573, U504 74LS573, U505 74LS573, U506 74LS573, U507 74LS573, U508 74LS573, U509 74LS573

Commit message: [pcb][tri-sram] tri-sram complete
squashed big-bus branch
Parts:
- renumbered C519 to C301, C503 to C302, C512 to C303, C521 to C304, C525 to C305, C506 to C306, C518 to C307, C527 to C308, C522 to C309, C509 to C310, C515 to C311, C524 to C312, U501 to U301, U504 to U302, U507 to U303, U502 to U304, U506 to U305, U509 to U306, U503 to U307, U505 to U308, U508 to U309
Connections:
- net 0_A1: now also U303.15 (Q4); no longer U303.12 (Q7)
- net 0_A2: now also U303.14 (Q5); no longer U303.13 (Q6)
- net 0_A3: now also U303.13 (Q6); no longer U303.14 (Q5)
- net 0_A4: now also U303.12 (Q7); no longer U303.15 (Q4)
- net 1_A1: now also U306.15 (Q4); no longer U306.12 (Q7)
- net 1_A2: now also U306.14 (Q5); no longer U306.13 (Q6)
- net 1_A3: now also U306.13 (Q6); no longer U306.14 (Q5)
- net 1_A4: now also U306.12 (Q7); no longer U306.15 (Q4)
- net 2_A1: now also U309.15 (Q4); no longer U309.12 (Q7)
- net 2_A2: now also U309.14 (Q5); no longer U309.13 (Q6)
- net 2_A3: now also U309.13 (Q6); no longer U309.14 (Q5)
- net 2_A4: now also U309.12 (Q7); no longer U309.15 (Q4)
- net A1: now also U303.6 (D4), U306.6 (D4), U309.6 (D4); no longer U303.9 (D7), U306.9 (D7), U309.9 (D7)
- net A10: now also U308.5 (D3); no longer U308.4 (D2)
- net A11: now also U308.6 (D4); no longer U308.5 (D3)
- net A12: now also U308.7 (D5); no longer U308.6 (D4)
- net A13: now also U308.8 (D6); no longer U308.7 (D5)
- net A14: now also U308.9 (D7); no longer U308.8 (D6)
- net A15: no longer U308.9 (D7)
- net A2: now also U303.7 (D5), U306.7 (D5), U309.7 (D5); no longer U303.8 (D6), U306.8 (D6), U309.8 (D6)
- net A3: now also U303.8 (D6), U306.8 (D6), U309.8 (D6); no longer U303.7 (D5), U306.7 (D5), U309.7 (D5)
- net A4: now also U303.9 (D7), U306.9 (D7), U309.9 (D7); no longer U303.6 (D4), U306.6 (D4), U309.6 (D4)
- net A7: now also U308.2 (D0)
- net A8: now also U308.3 (D1); no longer U308.2 (D0)
- net A9: now also U308.4 (D2); no longer U308.3 (D1)
Other:
- moved on the sheet: C305, C307, C308, U305, U306

Commit message: [pcb][tri-sram] add part numbers
Parts:
- U301, U302, U303, U304, U305, U306, U307, U308, U309: Digi-Key Part Number (none) -> 264-74LCX541FT(AE)CT-ND
Changed lines of the file:
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@@
+			)
+		)
+		(property "Digi-Key Part Number" "264-74LCX541FT(AE)CT-ND"
+			(at 59.69 135.89 0)
+			(effects
+				(font
+					(size 1.27 1.27)
+				)
+				(hide yes)
 			)
 		)
@@
 			)
 		)
+		(property "Digi-Key Part Number" "264-74LCX541FT(AE)CT-ND"
+			(at 251.46 195.58 0)
+			(effects
+				(font
+					(size 1.27 1.27)
+				)
+				(hide yes)
+			)
+		)
 		(pin "5"
 		)
@@
 			)
 		)
+		(property "Digi-Key Part Number" "264-74LCX541FT(AE)CT-ND"
+			(at 156.21 135.89 0)
+			(effects
+				(font
+					(size 1.27 1.27)
+				)
+				(hide yes)
+			)
+		)
 		(pin "5"
 		)
@@
 			)
 		)
+		(property "Digi-Key Part Number" "264-74LCX541FT(AE)CT-ND"
+			(at 251.46 135.89 0)
+			(effects
+				(font
+					(size 1.27 1.27)
+				)
+				(hide yes)
+			)
+		)
 		(pin "5"
 		)
@@
 			)
 		)
+		(property "Digi-Key Part Number" "264-74LCX541FT(AE)CT-ND"
+			(at 251.46 74.93 0)
+			(effects
+				(font
+					(size 1.27 1.27)
+				)
+				(hide yes)
+			)
+		)
 		(pin "5"
 		)
@@
 			)
 		)
+		(property "Digi-Key Part Number" "264-74LCX541FT(AE)CT-ND"
+			(at 59.69 74.93 0)
+			(effects
+				(font
+					(size 1.27 1.27)
+				)
+				(hide yes)
+			)
+		)
 		(pin "5"
 		)
@@
 			)
 		)
+		(property "Digi-Key Part Number" "264-74LCX541FT(AE)CT-ND"
+			(at 156.21 74.93 0)
+			(effects
+				(font
+					(size 1.27 1.27)
+				)
+				(hide yes)
+			)
+		)
 		(pin "5"
 		)
@@
 			)
 		)
+		(property "Digi-Key Part Number" "264-74LCX541FT(AE)CT-ND"
+			(at 59.69 195.58 0)
+			(effects
+				(font
+					(size 1.27 1.27)
+				)
+				(hide yes)
+			)
+		)
 		(pin "5"
 		)
@@
 			(at 156.21 195.58 0)
 			(effects
+				(font
+					(size 1.27 1.27)
+				)
+				(hide yes)
+			)
+		)
+		(property "Digi-Key Part Number" "264-74LCX541FT(AE)CT-ND"
+			(at 156.21 195.58 0)
+			(effects

Commit message: [pcb][3xsram] fix latch part number
Parts:
- U301, U302, U303, U304, U305, U306, U307, U308, U309: Digi-Key Part Number 264-74LCX541FT(AE)CT-ND -> 2156-74LS573SCX-ND; LCSC Part # C7194124 -> (none)
Changed lines of the file:
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@@
 			)
 		)
-		(property "LCSC Part #" "C7194124"
+		(property "LCSC Part #" ""
 			(at 59.69 135.89 0)
 			(effects
@@
 			)
 		)
-		(property "Digi-Key Part Number" "264-74LCX541FT(AE)CT-ND"
+		(property "Digi-Key Part Number" "2156-74LS573SCX-ND"
 			(at 59.69 135.89 0)
 			(effects
@@
 			)
 		)
-		(property "LCSC Part #" "C7194124"
+		(property "LCSC Part #" ""
 			(at 251.46 195.58 0)
 			(effects
@@
 			)
 		)
-		(property "Digi-Key Part Number" "264-74LCX541FT(AE)CT-ND"
+		(property "Digi-Key Part Number" "2156-74LS573SCX-ND"
 			(at 251.46 195.58 0)
 			(effects
@@
 			)
 		)
-		(property "LCSC Part #" "C7194124"
+		(property "LCSC Part #" ""
 			(at 156.21 135.89 0)
 			(effects
@@
 			)
 		)
-		(property "Digi-Key Part Number" "264-74LCX541FT(AE)CT-ND"
+		(property "Digi-Key Part Number" "2156-74LS573SCX-ND"
 			(at 156.21 135.89 0)
 			(effects
@@
 			)
 		)
-		(property "LCSC Part #" "C7194124"
+		(property "LCSC Part #" ""
 			(at 251.46 135.89 0)
 			(effects
@@
 			)
 		)
-		(property "Digi-Key Part Number" "264-74LCX541FT(AE)CT-ND"
+		(property "Digi-Key Part Number" "2156-74LS573SCX-ND"
 			(at 251.46 135.89 0)
 			(effects
@@
 			)
 		)
-		(property "LCSC Part #" "C7194124"
+		(property "LCSC Part #" ""
 			(at 251.46 74.93 0)
 			(effects
@@
 			)
 		)
-		(property "Digi-Key Part Number" "264-74LCX541FT(AE)CT-ND"
+		(property "Digi-Key Part Number" "2156-74LS573SCX-ND"
 			(at 251.46 74.93 0)
 			(effects
@@
 			)
 		)
-		(property "LCSC Part #" "C7194124"
+		(property "LCSC Part #" ""
 			(at 59.69 74.93 0)
 			(effects
@@
 			)
 		)
-		(property "Digi-Key Part Number" "264-74LCX541FT(AE)CT-ND"
+		(property "Digi-Key Part Number" "2156-74LS573SCX-ND"
 			(at 59.69 74.93 0)
 			(effects
@@
 			)
 		)
-		(property "LCSC Part #" "C7194124"
+		(property "LCSC Part #" ""
 			(at 156.21 74.93 0)
 			(effects
@@
 			)
 		)
-		(property "Digi-Key Part Number" "264-74LCX541FT(AE)CT-ND"
+		(property "Digi-Key Part Number" "2156-74LS573SCX-ND"
 			(at 156.21 74.93 0)
 			(effects
@@
 			)
 		)
-		(property "LCSC Part #" "C7194124"
+		(property "LCSC Part #" ""
 			(at 59.69 195.58 0)
 			(effects
@@
 			)
 		)
-		(property "Digi-Key Part Number" "264-74LCX541FT(AE)CT-ND"
+		(property "Digi-Key Part Number" "2156-74LS573SCX-ND"
 			(at 59.69 195.58 0)
 			(effects
@@
 			)
 		)
-		(property "LCSC Part #" "C7194124"
+		(property "LCSC Part #" ""
 			(at 156.21 195.58 0)
 			(effects
@@
 			)
 		)
-		(property "Digi-Key Part Number" "264-74LCX541FT(AE)CT-ND"
+		(property "Digi-Key Part Number" "2156-74LS573SCX-ND"
 			(at 156.21 195.58 0)
 			(effects
