File: pcb/vanilla-ice40/vanilla-ice40.kicad_sch (KiCad schematic)
At the start: 109 parts, among them J1 Conn_01x02_Pin, J2 SM04B-SRSS-TBLFSN, J3 FX18-120S-0.8SH, J4 Conn_01x06_Pin, J5 Conn_01x02_Pin, J6 Conn_01x02_Pin, J7 Conn_01x02_Pin, U1 TPS563252DRLR, U2 ICE40HX4K-TQ144, U3 W25X40CLSN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

Commit message: fix 1 off error in fx18 pin layout
Connections:
- net +3V3: now also J3.71, J3.81; no longer J3.70, J3.80
- net GND: now also J3.72, J3.82; no longer J3.71, J3.81
- net IOR_139: now also J3.80; no longer J3.82
- net IOR_160: now also J3.70; no longer J3.72
Changed lines of the file:
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@@
 	)
 	(label "IOR_139"
-		(at 254 182.88 0)
+		(at 254 187.96 0)
 		(fields_autoplaced yes)
 		(effects
@@
 	)
 	(label "+3V3"
-		(at 254 187.96 0)
+		(at 254 185.42 0)
 		(fields_autoplaced yes)
 		(effects
@@
 	)
 	(label "+3V3"
-		(at 254 213.36 0)
+		(at 254 210.82 0)
 		(fields_autoplaced yes)
 		(effects
@@
 	)
 	(label "GND"
-		(at 254 185.42 0)
+		(at 254 182.88 0)
 		(fields_autoplaced yes)
 		(effects
@@
 	)
 	(label "IOR_160"
-		(at 254 208.28 0)
+		(at 254 213.36 0)
 		(fields_autoplaced yes)
 		(effects
@@
 	)
 	(label "GND"
-		(at 254 210.82 0)
-		(fields_autoplaced yes)
-		(effects
+		(at 254 208.28 0)
+		(fields_autoplaced yes)
+		(effects

Commit message: [pcb] misc updates prior to ordder
Parts:
- removed 1V2_1, 3V3_1: Red, Diode_SMD:D_0603_1608Metric, symbol Device:LED_Small
- removed R11, R21: 2.2k, Resistor_SMD:R_0603_1608Metric, symbol Device:R_Small
- R6: value 2.2k -> 5.1k; Digi-Key Part Number 118-CR0603-FX-2201ELFCT-ND -> CR0603-FX-5101ELFCT-ND; LCSC Part # C4190 -> C23186
Connections:
- net VBUS_5V: now also R6.2, U1.5 (EN); no longer R6.1
- net at 5V_1.2 (A): now also R6.1; no longer R6.2
- no-connect marks 32 -> 31
