File: pcb/breakout-sram-256x2/breakout-sram-256x2.kicad_sch (KiCad schematic)
At the start: 10 parts, among them J1 FX18-120P-0.8SV20, J2 FX18-120S-0.8SV20, U1 IS61WV25616-10TLI, U3 IS61WV25616-10TLI

Commit message: [axi][sram] populate 256x2 part numbers
Parts:
- U1, U3: Digi-Key Part Number (none) -> 706-1146-ND; LCSC Part # (none) -> C883296
Changed lines of the file:
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@@
+			)
+		)
+		(property "LCSC Part #" "C883296"
+			(at 170.18 58.42 0)
+			(effects
+				(font
+					(size 1.27 1.27)
+				)
+				(hide yes)
+			)
+		)
+		(property "Digi-Key Part Number" "706-1146-ND"
+			(at 170.18 58.42 0)
+			(effects
+				(font
+					(size 1.27 1.27)
+				)
+				(hide yes)
 			)
 		)
@@
 			(at 171.45 172.72 0)
 			(effects
+				(font
+					(size 1.27 1.27)
+				)
+				(hide yes)
+			)
+		)
+		(property "LCSC Part #" "C883296"
+			(at 171.45 172.72 0)
+			(effects
+				(font
+					(size 1.27 1.27)
+				)
+				(hide yes)
+			)
+		)
+		(property "Digi-Key Part Number" "706-1146-ND"
+			(at 171.45 172.72 0)
+			(effects

Commit message: [axi][sram] set jlcpcb rotation
Parts:
- J2: JLCPCB Rotation Offset (none) -> 180
- U1, U3: JLCPCB Rotation Offset (none) -> -90
Changed lines of the file:
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@@
+			)
+		)
+		(property "JLCPCB Rotation Offset" "180"
+			(at 356.87 96.52 0)
+			(effects
+				(font
+					(size 1.27 1.27)
+				)
+				(hide yes)
 			)
 		)
@@
 			)
 		)
+		(property "JLCPCB Rotation Offset" "-90"
+			(at 170.18 58.42 0)
+			(effects
+				(font
+					(size 1.27 1.27)
+				)
+				(hide yes)
+			)
+		)
 		(pin "30"
 		)
@@
 			)
 		)
+		(property "JLCPCB Rotation Offset" "180"
+			(at 322.58 96.52 0)
+			(effects
+				(font
+					(size 1.27 1.27)
+				)
+				(hide yes)
+			)
+		)
 		(pin "117"
 		)
@@
 			)
 		)
+		(property "JLCPCB Rotation Offset" "-90"
+			(at 171.45 172.72 0)
+			(effects
+				(font
+					(size 1.27 1.27)
+				)
+				(hide yes)
+			)
+		)
 		(pin "30"
 		)
@@
 			(at 393.7 96.52 0)
 			(effects
+				(font
+					(size 1.27 1.27)
+				)
+				(hide yes)
+			)
+		)
+		(property "JLCPCB Rotation Offset" "180"
+			(at 393.7 96.52 0)
+			(effects
