File: pcb/breakout-adc/b2b.kicad_sch (KiCad schematic)
At the start: 5 parts, among them J27 DF40C-100DP-0.4V51, J28 DF40C-100DP-0.4V51, J29 DF40C-100DP-0.4V51, J30 DF40C-100DP-0.4V51, J32 DF40C-40DP-0.4V51

Commit message: [adc][sram] fix part numbers for plugs
Parts:
- J27, J28, J29, J30: LCSC Part # C597931 -> C531031
Changed lines of the file:
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@@
 			)
 		)
-		(property "LCSC Part #" "C597931"
+		(property "LCSC Part #" "C531031"
 			(at 240.03 87.63 0)
 			(effects
@@
 			)
 		)
-		(property "LCSC Part #" "C597931"
+		(property "LCSC Part #" "C531031"
 			(at 293.37 87.63 0)
 			(effects
@@
 			)
 		)
-		(property "LCSC Part #" "C597931"
+		(property "LCSC Part #" "C531031"
 			(at 341.63 87.63 0)
 			(effects
@@
 			)
 		)
-		(property "LCSC Part #" "C597931"
+		(property "LCSC Part #" "C531031"
 			(at 389.89 87.63 0)
 			(effects
