File: pcb/vanilla-ice40-8k/vanilla-ice40-8k.kicad_sch (KiCad schematic)
At the start: 17 parts, among them J1 QSH-060-01-L-D-A, J2 QSH-060-01-L-D-A, J3 QTH-060-01-L-D-A, J4 QTH-060-01-L-D-A, U1 ICE40HX8K-CT256, X1 SG-8101CE 100Mhz

Commit message: [hx8k][pcb] move headers and banks to sheets
Parts:
- removed J1, J2: QSH-060-01-L-D-A, !Misc:SAMTEC_QSH-060-01-X-D-A, symbol !Misc:QSH-060-01-L-D-A
- removed J3, J4: QTH-060-01-L-D-A, !Misc:SAMTEC_QTH-060-01-X-D-A, symbol !Misc:QTH-060-01-L-D-A
- removed U1: ICE40HX8K-CT256, ICE40HX8K-CT256:BGA256C80P16X16_1400X1400X170, symbol ICE40HX8K-CT256:ICE40HX8K-CT256
Other:
- added sheet headers (headers.kicad_sch)
- added sheet hx8k banks (hx8k_banks.kicad_sch)
- note removed: "44+2+3 = 49"
- note removed: "50"
- note removed: "51"
- note removed: "52"
- moved on the sheet: R3, USR1
