File: pcb/vanilla-ice40-8k/hx8k_power.kicad_sch (KiCad schematic)
At the start: 36 parts, among them U1 ICE40HX8K-CT256

Commit message: [hx8k][pcb] move usb_c_power to use symbol lib
Parts:
- C10, C12, C15, C2, C20, C25, C30: symbol Device:C_Small -> !Misc:C_22uf_0603; LCSC Part # C59461 -> C59461
Changed lines of the file:
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@@
 	)
 	(symbol
-		(lib_id "Device:C_Small")
+		(lib_id "!Misc:C_22uf_0603")
 		(at 162.56 86.36 0)
 		(unit 1)
@@
 			)
 		)
-		(property "Description" "Unpolarized capacitor, small symbol"
+		(property "Description" "Unpolarized capacitor 22uf 0603 6.3V"
 			(at 162.56 86.36 0)
 			(effects
@@
 			)
 		)
-		(property "LCSC Part #" "C59461"
+		(property "LCSC Part #" " C59461"
 			(at 162.56 86.36 0)
 			(effects
@@
 	)
 	(symbol
-		(lib_id "Device:C_Small")
+		(lib_id "!Misc:C_22uf_0603")
 		(at 163.83 49.53 0)
 		(unit 1)
@@
 			)
 		)
-		(property "Description" "Unpolarized capacitor, small symbol"
+		(property "Description" "Unpolarized capacitor 22uf 0603 6.3V"
 			(at 163.83 49.53 0)
 			(effects
@@
 			)
 		)
-		(property "LCSC Part #" "C59461"
+		(property "LCSC Part #" " C59461"
 			(at 163.83 49.53 0)
 			(effects
@@
 	)
 	(symbol
-		(lib_id "Device:C_Small")
+		(lib_id "!Misc:C_22uf_0603")
 		(at 38.1 115.57 0)
 		(unit 1)
@@
 			)
 		)
-		(property "Description" "Unpolarized capacitor, small symbol"
+		(property "Description" "Unpolarized capacitor 22uf 0603 6.3V"
 			(at 38.1 115.57 0)
 			(effects
@@
 			)
 		)
-		(property "LCSC Part #" "C59461"
+		(property "LCSC Part #" " C59461"
 			(at 38.1 115.57 0)
 			(effects
@@
 	)
 	(symbol
-		(lib_id "Device:C_Small")
+		(lib_id "!Misc:C_22uf_0603")
 		(at 162.56 115.57 0)
 		(unit 1)
@@
 			)
 		)
-		(property "Description" "Unpolarized capacitor, small symbol"
+		(property "Description" "Unpolarized capacitor 22uf 0603 6.3V"
 			(at 162.56 115.57 0)
 			(effects
@@
 			)
 		)
-		(property "LCSC Part #" "C59461"
+		(property "LCSC Part #" " C59461"
 			(at 162.56 115.57 0)
 			(effects
@@
 	)
 	(symbol
-		(lib_id "Device:C_Small")
+		(lib_id "!Misc:C_22uf_0603")
 		(at 186.69 49.53 0)
 		(unit 1)
@@
 			)
 		)
-		(property "Description" "Unpolarized capacitor, small symbol"
+		(property "Description" "Unpolarized capacitor 22uf 0603 6.3V"
 			(at 186.69 49.53 0)
 			(effects
@@
 			)
 		)
-		(property "LCSC Part #" "C59461"
+		(property "LCSC Part #" " C59461"
 			(at 186.69 49.53 0)
 			(effects
@@
 	)
 	(symbol
-		(lib_id "Device:C_Small")
+		(lib_id "!Misc:C_22uf_0603")
 		(at 38.1 48.26 0)
 		(unit 1)
@@
 			)
 		)
-		(property "Description" "Unpolarized capacitor, small symbol"
+		(property "Description" "Unpolarized capacitor 22uf 0603 6.3V"
 			(at 38.1 48.26 0)
 			(effects
@@
 			)
 		)
-		(property "LCSC Part #" "C59461"
+		(property "LCSC Part #" " C59461"
 			(at 38.1 48.26 0)
 			(effects
@@
 	)
 	(symbol
-		(lib_id "Device:C_Small")
+		(lib_id "!Misc:C_22uf_0603")
 		(at 38.1 86.36 0)
 		(unit 1)
@@
 			)
 		)
-		(property "Description" "Unpolarized capacitor, small symbol"
+		(property "Description" "Unpolarized capacitor 22uf 0603 6.3V"
 			(at 38.1 86.36 0)
 			(effects
@@
 			)
 		)
-		(property "LCSC Part #" "C59461"
+		(property "LCSC Part #" " C59461"
 			(at 38.1 86.36 0)
 			(effects
