File: pcb/vanilla-ice40-8k/sram_programmer.kicad_sch (KiCad schematic)
At the start: 32 parts, among them U2 W25X40CLSN, U3 FT2232HQ, U4 93LCxxBxxOT, Y1 12Mhz/18pf

Commit message: [hx8k][pcb] part cleanup
Parts:
- FB1, FB2: value 600ohm/200ma -> 600/200ma
- R18, R20, R21, R22, R23, R26, R27, R28: value 10k -> 10K
- R19: value 12k -> 12K
- R29: value 2.2k -> 2.2K
- Y1: value 12Mhz/18pf -> 12MHz/20pf
