File: pcb/sram-256x4/interim.kicad_sch (KiCad schematic)
At the start: 7 parts

Commit message: [pcb][sram-4x] fully routed
Parts:
- removed PM1, PM2: Conn_02x06_Top_Bottom, custom:PMOD_12p_Horizontal, symbol Connector_Generic:Conn_02x06_Top_Bottom
Connections:
- net C_58 renamed C23
- net C_62 renamed C25
- net C_66 renamed C27
- net C_70 renamed C29
- net C_74 renamed C31
- net C_78 renamed C33
- net C_82 renamed C35
- net C_86 renamed C37
- net C_90 renamed D25
- net C_94 renamed D29
- net C_98 renamed D27
- net D_20 renamed D31
- net D_24 renamed D33
- net D_28 renamed D35
- no-connect marks 189 -> 187
Other:
- note added: "PM1_1"
- note added: "PM1_10"
- note added: "PM1_2"
- note added: "PM1_3"
- note added: "PM1_4"
- note added: "PM1_7"
- note added: "PM1_8"
- note added: "PM1_9"
- note added: "PM2_1"
- note added: "PM2_2"
- note added: "PM2_3"
- note added: "PM2_4"
- note added: "PM2_7"
- note added: "PM2_8"
- moved on the sheet: JL3
